File: cpu/Controls/ControlModule.sch (KiCad schematic (older format))
At the start: 19 parts, among them J1 Interconnect, SW1 SW_SPST, SW2 SW_SPST, SW3 SW_SPST, SW4 SW_SPST, U1 74LS14

Commit message: Lots of changes
Parts:
- added C4: 1uF, Capacitor_SMD:CP_Elec_4x5.4, symbol Device:CP
- added C5: 0.1uF, Capacitor_SMD:C_0603_1608Metric_Pad1.05x0.95mm_HandSolder, symbol Device:C
- added D4: 1N4148, Diode_SMD:D_SOD-523, symbol Device:D
- added R7: 82K, Resistor_SMD:R_0603_1608Metric_Pad1.05x0.95mm_HandSolder, symbol Device:R
- added R8: 20K, Resistor_SMD:R_0603_1608Metric_Pad1.05x0.95mm_HandSolder, symbol Device:R
- added SW5: SW_SPST, Button_Switch_THT:SW_PUSH_6mm_H5mm, symbol Switch:SW_SPST
- C1, C2, C3: footprint Capacitor_SMD:C_0603_1608Metric_Pad1.05x0.95mm_HandSolder -> Capacitor_SMD:CP_Elec_4x5.4; symbol Device:C -> Device:CP; Digikey (none) -> 493-9795-1-ND
- J1: footprint (none) -> Connector_PinHeader_2.54mm:PinHeader_2x17_P2.54mm_Horizontal; Digikey (none) -> S5531-ND
- POT1: Digikey (none) -> 987-1710-ND
- SW1, SW3: footprint (none) -> Button_Switch_THT:SW_PUSH_6mm_H5mm; Digikey (none) -> EG1861-ND
- SW2, SW4: footprint (none) -> Button_Switch_THT:SW_PUSH_6mm_H5mm; Digikey (none) -> 401-1132-ND
Connections:
- net labels added: CLK, DBG, RST, ~CLK
- wire segments 68 -> 91
- no-connect marks 8 -> 26
Other:
- note added: "Reset Switch\n(debounced)"
- moved on the sheet: U1D
