File: cpu/Controls/ControlModule.kicad_pcb (KiCad board)
At the start: 2 copper layers, 14 parts, among them U1 74LS14

Commit message: Lots of changes
Parts:
- added C4: 1uF, Capacitor_SMD:CP_Elec_4x5.4, F.Cu at (213.8, 34.0)
- added C5: 0.1uF, Capacitor_SMD:C_0603_1608Metric_Pad1.05x0.95mm_HandSolder, F.Cu at (142.0, 41.0)
- added D4: 1N4148, Diode_SMD:D_SOD-523, F.Cu at (213.0, 41.0)
- added J1: Interconnect, Connector_PinHeader_2.54mm:PinHeader_2x17_P2.54mm_Horizontal, F.Cu at (184.0, 80.0)
- added R7: 82K, Resistor_SMD:R_0603_1608Metric_Pad1.05x0.95mm_HandSolder, F.Cu at (212.1, 45.0)
- added R8: 20K, Resistor_SMD:R_0603_1608Metric_Pad1.05x0.95mm_HandSolder, F.Cu at (212.1, 52.0)
- added SW1: SW_SPST, Button_Switch_THT:SW_PUSH_6mm_H5mm, F.Cu at (107.0, 21.0)
- added SW2: SW_SPST, Button_Switch_THT:SW_PUSH_6mm_H5mm, F.Cu at (117.3, 21.0)
- added SW3: SW_SPST, Button_Switch_THT:SW_PUSH_6mm_H5mm, F.Cu at (200.0, 22.0)
- added SW4: SW_SPST, Button_Switch_THT:SW_PUSH_6mm_H5mm, F.Cu at (222.0, 21.5)
- added SW5: SW_SPST, Button_Switch_THT:SW_PUSH_6mm_H5mm, F.Cu at (211.0, 21.5)
- C1, C2, C3: footprint Capacitor_SMD:C_0603_1608Metric_Pad1.05x0.95mm_HandSolder -> Capacitor_SMD:CP_Elec_4x5.4
- moved C3 81.3 mm to (203.0, 34.0)
- moved R5 76.4 mm to (202.1, 47.0)
- moved R6 70.3 mm to (202.1, 51.0)
- moved D3 68.7 mm to (202.3, 42.0)
- moved POT1 64.1 mm to (169.0, 34.0)
- moved D1 41.3 mm to (108.3, 36.0)
- moved C1 41.3 mm to (110.0, 31.0)
- moved R2 35.9 mm to (112.0, 39.0)
- moved R1 35.2 mm to (112.1, 36.0)
- moved D2 34.9 mm to (117.7, 36.0)
- moved C2 31.5 mm to (120.5, 31.0)
- moved R3 31.1 mm to (121.1, 36.0)
- moved R4 23.8 mm to (121.1, 47.0)
- moved U1 13.8 mm to (140.7, 50.0)
Connections:
- POT1 pad 2: SPD1 -> /SPD1
- POT1 pad 3: SPD2 -> /SPD2
- U1 pad 2: MAN -> /MAN
- U1 pad 4: SEL -> /SEL
- U1 pad 6: SEL -> /HLT
- U1 pad 8: Net-(U1-Pad8) -> /RST
Other:
- board outline added: 125 x 50 mm

Commit message: Upgrade to KiCad 6 and commit a bunch of random stuff
Connections:
- net /~CLK renamed /~{CLK}
Other:
- net class Default removed
