File: cpu/CounterRegister/CounterRegisterModule.sch (KiCad schematic (older format))
At the start: 0 parts

Commit message: Lots of changes
Parts:
- added C1, C10, C11, C12, C2, C3, C4, C5, C6, C7, C8, C9: 0.1uF, Capacitor_SMD:C_0603_1608Metric_Pad1.05x0.95mm_HandSolder, symbol Device:C
- added D1, D10, D11, D12, D13, D14, D15, D16, D2, D3, D4, D5, D6, D7, D8, D9: D_RED, LED_SMD:LED_1206_3216Metric_Pad1.42x1.75mm_HandSolder, symbol Device:D_ALT
- added D17, D18, D19, D20, D21, D22, D23: D_AMBER, LED_SMD:LED_1206_3216Metric_Pad1.42x1.75mm_HandSolder, symbol Device:D_ALT
- added J1: Interconnect A, Connector_PinHeader_2.54mm:PinHeader_2x17_P2.54mm_Horizontal, symbol Connector_Generic:Conn_02x17_Odd_Even
- added J2: Interconnect B, Connector_PinHeader_2.54mm:PinHeader_2x17_P2.54mm_Horizontal, symbol Connector_Generic:Conn_02x17_Odd_Even
- added R1, R10, R11, R12, R13, R14, R15, R16, R17, R18, R19, R2, R20, R21, R22, R23, R3, R4, R5, R6, R7, R8, R9: 220R, Resistor_SMD:R_0603_1608Metric_Pad1.05x0.95mm_HandSolder, symbol Device:R
- added U1, U2, U3, U4: 74LS193, Package_SO:SOIC-16_3.9x9.9mm_P1.27mm, symbol 74xx:74LS193
- added U10, U11, U5, U6, U7, U8, U9: 74LS245, symbol 74ls245_bidirection:74LS245_BiDirection
- added U12: 74LS00, Package_SO:SOIC-14_3.9x8.7mm_P1.27mm, symbol 74xx:74LS00
Connections:
- net labels added: +5V, CLK, GND, HLT, RST, a_bus_00, a_bus_01, a_bus_02, a_bus_03, a_bus_04, a_bus_05, a_bus_06, a_bus_07, a_bus_08, a_bus_09, a_bus_10, a_bus_11, a_bus_12, a_bus_13, a_bus_14, a_bus_15, a_bus_write, d_bus_00, d_bus_01, d_bus_02, d_bus_03, d_bus_04, d_bus_05, d_bus_06, d_bus_07, d_bus_08, d_bus_09, d_bus_10, d_bus_11, d_bus_12, d_bus_13, d_bus_14, d_bus_15, d_bus_read, d_bus_write, reg_00, reg_01, reg_02, reg_03, reg_04, reg_05, reg_06, reg_07, reg_08, reg_09, reg_10, reg_11, reg_12, reg_13, reg_14, reg_15, reg_borrow, reg_carry, reg_dec, reg_inc, ~CLK, ~DBG, ~a_bus_write_CLK, ~d_bus_read, ~d_bus_write_CLK
- wire segments 0 -> 532
- no-connect marks 0 -> 27
Other:
- note added: "Address Bus"
- note added: "Data Bus"
