File: cpu/CounterRegister/CounterRegisterModule.sch (KiCad schematic (older format))
At the start: 72 parts, among them J1 Interconnect A, J2 Interconnect B, U1 74LS193, U10 74LS245, U11 74LS245, U12 74LS00, U2 74LS193, U3 74LS193, U4 74LS193, U5 74LS245, U6 74LS245, U7 74LS245, U8 74LS245, U9 74LS245

Commit message: Completed GPR 1.2 PCB and started lots of other things. * Started ALU * Updated Constant Reg * Completed v1.2 GPR * Added random symbols * Updated Memory * Updated plots
Parts:
- removed J1: Interconnect A, Connector_PinHeader_2.54mm:PinHeader_2x17_P2.54mm_Horizontal, symbol Connector_Generic:Conn_02x17_Odd_Even
- removed J2: Interconnect B, Connector_PinHeader_2.54mm:PinHeader_2x17_P2.54mm_Horizontal, symbol Connector_Generic:Conn_02x17_Odd_Even
- added J1: Interconnect, Connector_PCBEdge:BUS_PCI, symbol MySymbols:Bus_PCI_32bit_5V
- D11, D12, D13, D14, D15, D16: symbol Device:D_ALT -> Device:LED_ALT
- U10, U11, U5, U6, U7, U8, U9: footprint (none) -> Package_SO:SOIC-20W_7.5x12.8mm_P1.27mm; symbol 74ls245_bidirection:74LS245_BiDirection -> CounterRegisterModule-rescue:74LS245_BiDirection-74ls245_bidirection
Connections:
- wire segments 532 -> 540
- no-connect marks 27 -> 75
Other:
- moved on the sheet: D1, D10, D17, D18, D19, D2, D20, D21, D22, D23, D3, D4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
