File: cpu/CounterRegister/CounterRegisterModule.kicad_pcb (KiCad board)
At the start: 2 copper layers, 139.7 x 64.3 mm, 67 parts, among them J1 Interconnect 1, J2 Interconnect 2, U1 74HCT574, U10 74LS245, U11 74LS245, U12 74LS245, U13 74LS126, U2 74HCT574, U3 74LS14, U5 74LS245, U6 74LS245, U7 74LS245, U8 74LS245, U9 74LS245

Commit message: Lots of changes
Parts:
- removed C13: 0.1uF, Capacitor_SMD:C_0603_1608Metric_Pad1.05x0.95mm_HandSolder
- removed D0: LED_RED, LED_SMD:LED_1206_3216Metric_Pad1.42x1.75mm_HandSolder
- removed R0: 220R, Resistor_SMD:R_0603_1608Metric_Pad1.05x0.95mm_HandSolder
- removed U13: 74LS126, Package_SO:SOIC-14_3.9x8.7mm_P1.27mm
- added D20: D_AMBER, LED_SMD:LED_1206_3216Metric_Pad1.42x1.75mm_HandSolder, F.Cu at (169.8, 111.2)
- added D21: D_AMBER, LED_SMD:LED_1206_3216Metric_Pad1.42x1.75mm_HandSolder, F.Cu at (163.8, 114.6)
- added D22: D_AMBER, LED_SMD:LED_1206_3216Metric_Pad1.42x1.75mm_HandSolder, F.Cu at (181.8, 74.5)
- added D23: D_AMBER, LED_SMD:LED_1206_3216Metric_Pad1.42x1.75mm_HandSolder, F.Cu at (181.8, 71.1)
- added R20: 220R, Resistor_SMD:R_0603_1608Metric_Pad1.05x0.95mm_HandSolder, F.Cu at (183.6, 82.4)
- added R21: 220R, Resistor_SMD:R_0603_1608Metric_Pad1.05x0.95mm_HandSolder, F.Cu at (164.8, 120.0)
- added R22: 220R, Resistor_SMD:R_0603_1608Metric_Pad1.05x0.95mm_HandSolder, F.Cu at (160.5, 124.7)
- added R23: 220R, Resistor_SMD:R_0603_1608Metric_Pad1.05x0.95mm_HandSolder, F.Cu at (145.9, 107.5)
- added U4: 74LS193, Package_SO:SOIC-16_3.9x9.9mm_P1.27mm, F.Cu at (105.7, 82.0)
- D1, D10, D11, D12, D13, D14, D15, D2, D3, D4, D5, D6, D7, D8, D9: value LED_RED -> D_RED
- D16: value LED_AMBER -> D_RED
- D17, D18, D19: value LED_AMBER -> D_AMBER
- J1: value Interconnect 1 -> Interconnect A
- J2: value Interconnect 2 -> Interconnect B
- U1, U2: value 74HCT574 -> 74LS193; footprint Package_SO:SOIC-20W_7.5x12.8mm_P1.27mm -> Package_SO:SOIC-16_3.9x9.9mm_P1.27mm
- U12: value 74LS245 -> 74LS00; footprint Package_SO:SOIC-20W_7.5x12.8mm_P1.27mm -> Package_SO:SOIC-14_3.9x8.7mm_P1.27mm
- U3: value 74LS14 -> 74LS193; footprint Package_SO:SOIC-14_3.9x8.7mm_P1.27mm -> Package_SO:SOIC-16_3.9x9.9mm_P1.27mm
- moved D6 296.0 mm to (29.1, 85.1)
- moved D7 277.2 mm to (35.1, 88.5)
- moved C8 267.7 mm to (56.5, 89.2)
- moved D5 260.7 mm to (23.1, 88.5)
- moved D8 253.3 mm to (59.0, 86.2)
- moved C6 250.8 mm to (60.9, 89.2)
- moved D12 242.8 mm to (47.1, 88.5)
- moved C10 242.1 mm to (52.2, 89.2)
- moved D16 239.8 mm to (23.1, 85.1)
- moved D11 236.3 mm to (55.0, 82.9)
- moved D13 231.8 mm to (53.0, 86.2)
- moved D4 226.9 mm to (29.1, 88.5)
- moved D10 225.2 mm to (61.0, 82.9)
- moved D14 221.0 mm to (41.1, 88.5)
- moved U3 220.8 mm to (105.7, 70.5)
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Connections:
- C1 pad 1: +5V -> GND
- C1 pad 2: GND -> +5V
- C10 pad 1: +5V -> GND
- C10 pad 2: GND -> +5V
- C11 pad 1: +5V -> GND
- C11 pad 2: GND -> +5V
- C12 pad 1: +5V -> GND
- C12 pad 2: GND -> +5V
- C2 pad 1: +5V -> GND
- C2 pad 2: GND -> +5V
- C3 pad 1: +5V -> GND
- C3 pad 2: GND -> +5V
- C4 pad 1: +5V -> GND
- C4 pad 2: GND -> +5V
- C5 pad 1: +5V -> GND
- C5 pad 2: GND -> +5V
- C6 pad 1: +5V -> GND
- C6 pad 2: GND -> +5V
- C7 pad 1: +5V -> GND
- C7 pad 2: GND -> +5V
- C8 pad 1: +5V -> GND
- C8 pad 2: GND -> +5V
- C9 pad 1: +5V -> GND
- C9 pad 2: GND -> +5V
- D1 pad 2: /display_01 -> Net-(D1-Pad2)
- D10 pad 2: /display_10 -> Net-(D10-Pad2)
- D11 pad 2: /display_11 -> Net-(D11-Pad2)
- D12 pad 2: /display_12 -> Net-(D12-Pad2)
- D13 pad 2: /display_13 -> Net-(D13-Pad2)
- D14 pad 2: /display_14 -> Net-(D14-Pad2)
- D15 pad 2: /display_15 -> Net-(D15-Pad2)
- D2 pad 2: /display_02 -> Net-(D2-Pad2)
- D3 pad 2: /display_03 -> Net-(D3-Pad2)
- D4 pad 2: /display_04 -> Net-(D4-Pad2)
- D5 pad 2: /display_05 -> Net-(D5-Pad2)
- D6 pad 2: /display_06 -> Net-(D6-Pad2)
- D7 pad 2: /display_07 -> Net-(D7-Pad2)
- D8 pad 2: /display_08 -> Net-(D8-Pad2)
- D9 pad 2: /display_09 -> Net-(D9-Pad2)
- J1 pad 11: Net-(J1-Pad11) -> /reg_carry
- J1 pad 13: Net-(J1-Pad13) -> /reg_borrow
- J1 pad 25: /~DBG -> /DBG
- J1 pad 5: /x_bus_write -> /a_bus_write
- J1 pad 7: /y_bus_write -> /reg_inc
- J1 pad 9: Net-(J1-Pad9) -> /reg_dec
- J2 pad 1: /x_bus_15 -> Net-(J2-Pad1)
- J2 pad 10: /y_bus_11 -> /a_bus_11
- J2 pad 11: /x_bus_10 -> Net-(J2-Pad11)
- J2 pad 12: /y_bus_10 -> /a_bus_10
- J2 pad 13: /x_bus_09 -> Net-(J2-Pad13)
- J2 pad 14: /y_bus_09 -> /a_bus_09
- J2 pad 15: /x_bus_08 -> Net-(J2-Pad15)
- J2 pad 16: /y_bus_08 -> /a_bus_08
- J2 pad 17: /x_bus_07 -> Net-(J2-Pad17)
- J2 pad 18: /y_bus_07 -> /a_bus_07
- J2 pad 19: /x_bus_06 -> Net-(J2-Pad19)
- J2 pad 2: /y_bus_15 -> /a_bus_15
- J2 pad 20: /y_bus_06 -> /a_bus_06
- J2 pad 21: /x_bus_05 -> Net-(J2-Pad21)
- J2 pad 22: /y_bus_05 -> /a_bus_05
- J2 pad 23: /x_bus_04 -> Net-(J2-Pad23)
- J2 pad 24: /y_bus_04 -> /a_bus_04
- J2 pad 25: /x_bus_03 -> Net-(J2-Pad25)
- J2 pad 26: /y_bus_03 -> /a_bus_03
- J2 pad 27: /x_bus_02 -> Net-(J2-Pad27)
- J2 pad 28: /y_bus_02 -> /a_bus_02
- J2 pad 29: /x_bus_01 -> Net-(J2-Pad29)
- J2 pad 3: /x_bus_14 -> Net-(J2-Pad3)
- J2 pad 30: /y_bus_01 -> /a_bus_01
- J2 pad 31: /x_bus_00 -> Net-(J2-Pad31)
- J2 pad 32: /y_bus_00 -> /a_bus_00
- J2 pad 4: /y_bus_14 -> /a_bus_14
- J2 pad 5: /x_bus_13 -> Net-(J2-Pad5)
- J2 pad 6: /y_bus_13 -> /a_bus_13
- J2 pad 7: /x_bus_12 -> Net-(J2-Pad7)
- J2 pad 8: /y_bus_12 -> /a_bus_12
- J2 pad 9: /x_bus_11 -> Net-(J2-Pad9)
- R17 pad 2: GND -> Net-(R17-Pad2)
- R18 pad 2: GND -> Net-(R17-Pad2)
- R19 pad 2: GND -> Net-(R17-Pad2)
- U1 pad 1: GND -> /d_bus_01
- U1 pad 10: GND -> /d_bus_02
- U1 pad 12: /reg_07 -> Net-(U1-Pad12)
- U1 pad 13: /reg_06 -> Net-(U1-Pad13)
- U1 pad 14: /reg_05 -> /~RST
- U1 pad 15: /reg_04 -> /d_bus_00
- U1 pad 16: /reg_03 -> +5V
- U1 pad 2: /d_bus_00 -> /reg_01
- U1 pad 3: /d_bus_01 -> /reg_00
- U1 pad 4: /d_bus_02 -> /reg_dec
- U1 pad 5: /d_bus_03 -> /reg_inc
- U1 pad 6: /d_bus_04 -> /reg_02
- U1 pad 7: /d_bus_05 -> /reg_03
- U1 pad 8: /d_bus_06 -> GND
- U1 pad 9: /d_bus_07 -> /d_bus_03
- U10 pad 12: /reg_14 -> /reg_06
- U10 pad 13: /reg_13 -> /reg_05
- U10 pad 14: /reg_12 -> /reg_04
- U10 pad 15: /reg_11 -> /reg_03
- U10 pad 16: /reg_10 -> /reg_02
- U10 pad 17: /reg_09 -> /reg_01
- U10 pad 18: /reg_08 -> /reg_00
- U10 pad 19: /~y_bus_write -> /DBG
- U10 pad 2: /y_bus_08 -> Net-(D9-Pad2)
- U10 pad 3: /y_bus_09 -> Net-(D10-Pad2)
- U10 pad 4: /y_bus_10 -> Net-(D11-Pad2)
- U10 pad 5: /y_bus_11 -> Net-(D12-Pad2)
- U10 pad 6: /y_bus_12 -> Net-(D13-Pad2)
- U10 pad 7: /y_bus_13 -> Net-(D14-Pad2)
- U10 pad 8: /y_bus_14 -> Net-(D15-Pad2)
- U10 pad 9: /y_bus_15 -> Net-(D16-Pad2)
- U11 pad 11: /reg_07 -> Net-(U11-Pad11)
- U11 pad 12: /reg_06 -> /reg_borrow
- U11 pad 13: /reg_05 -> /reg_carry
- U11 pad 14: /reg_04 -> /reg_dec
- U11 pad 15: /reg_03 -> /reg_inc
- U11 pad 16: /reg_02 -> /a_bus_write
- U11 pad 17: /reg_01 -> /d_bus_write
- U11 pad 18: /reg_00 -> /d_bus_read
- U11 pad 19: /~DBG -> /DBG
- U11 pad 2: /display_00 -> Net-(D17-Pad2)
- U11 pad 3: /display_01 -> Net-(D18-Pad2)
- U11 pad 4: /display_02 -> Net-(D19-Pad2)
- U11 pad 5: /display_03 -> Net-(D20-Pad2)
- U11 pad 6: /display_04 -> Net-(D21-Pad2)
- U11 pad 7: /display_05 -> Net-(D22-Pad2)
- U11 pad 8: /display_06 -> Net-(D23-Pad2)
- U11 pad 9: /display_07 -> Net-(U11-Pad9)
- U12 pad 1: GND -> /RST
- U12 pad 10: GND -> /d_bus_write
- U12 pad 11: /reg_07 -> Net-(U12-Pad11)
- U12 pad 12: /reg_14 -> Net-(U12-Pad12)
- U12 pad 13: /reg_13 -> Net-(U12-Pad13)
- U12 pad 14: /reg_12 -> +5V
- U12 pad 2: /display_08 -> /RST
- U12 pad 3: /display_09 -> /~RST
- U12 pad 4: /display_10 -> /CLK
- U12 pad 5: /display_11 -> /a_bus_write
- U12 pad 6: /display_12 -> Net-(U12-Pad6)
- U12 pad 7: /display_13 -> GND
- U12 pad 8: /display_14 -> Net-(U12-Pad8)
- U12 pad 9: /display_15 -> /CLK
- U2 pad 1: GND -> /d_bus_05
- U2 pad 10: GND -> /d_bus_06
- U2 pad 12: /reg_07 -> Net-(U2-Pad12)
- U2 pad 13: /reg_14 -> Net-(U2-Pad13)
- U2 pad 14: /reg_13 -> /~RST
- U2 pad 15: /reg_12 -> /d_bus_04
- U2 pad 16: /reg_11 -> +5V
- U2 pad 2: /d_bus_08 -> /reg_05
- U2 pad 3: /d_bus_09 -> /reg_04
- U2 pad 4: /d_bus_10 -> Net-(U1-Pad13)
- U2 pad 5: /d_bus_11 -> Net-(U1-Pad12)
- U2 pad 6: /d_bus_12 -> /reg_06
- U2 pad 7: /d_bus_13 -> /reg_07
- U2 pad 8: /d_bus_14 -> GND
- U2 pad 9: /d_bus_15 -> /d_bus_07
- U3 pad 1: /d_bus_write -> /d_bus_09
- U3 pad 10: Net-(U3-Pad10) -> /d_bus_10
- U3 pad 11: Net-(U3-Pad11) -> /d_bus_read
- U3 pad 14: +5V -> /~RST
- U3 pad 2: /~d_bus_write -> /reg_09
- U3 pad 3: /x_bus_write -> /reg_08
- U3 pad 4: /~x_bus_write -> Net-(U2-Pad13)
- U3 pad 5: /y_bus_write -> Net-(U2-Pad12)
- U3 pad 6: /~y_bus_write -> /reg_10
- U3 pad 7: GND -> /reg_11
- U3 pad 8: Net-(U3-Pad8) -> GND
- U3 pad 9: Net-(U3-Pad9) -> /d_bus_11
- U5 pad 1: GND -> +5V
- U5 pad 11: /reg_07 -> /d_bus_07
- U5 pad 12: /reg_06 -> /d_bus_06
- U5 pad 13: /reg_05 -> /d_bus_05
- U5 pad 14: /reg_04 -> /d_bus_04
- U5 pad 15: /reg_03 -> /d_bus_03
- U5 pad 16: /reg_02 -> /d_bus_02
- U5 pad 17: /reg_01 -> /d_bus_01
- U5 pad 18: /reg_00 -> /d_bus_00
- U5 pad 19: /~d_bus_write -> Net-(U12-Pad8)
- U5 pad 2: /d_bus_00 -> /reg_00
- U5 pad 3: /d_bus_01 -> /reg_01
- U5 pad 4: /d_bus_02 -> /reg_02
- U5 pad 5: /d_bus_03 -> /reg_03
- U5 pad 6: /d_bus_04 -> /reg_04
- U5 pad 7: /d_bus_05 -> /reg_05
- U5 pad 8: /d_bus_06 -> /reg_06
- U5 pad 9: /d_bus_07 -> /reg_07
- U6 pad 1: GND -> +5V
- U6 pad 11: /reg_07 -> /d_bus_15
- U6 pad 12: /reg_14 -> /d_bus_14
- U6 pad 13: /reg_13 -> /d_bus_13
- U6 pad 14: /reg_12 -> /d_bus_12
- U6 pad 15: /reg_11 -> /d_bus_11
- U6 pad 16: /reg_10 -> /d_bus_10
- U6 pad 17: /reg_09 -> /d_bus_09
- U6 pad 18: /reg_08 -> /d_bus_08
- U6 pad 19: /~d_bus_write -> Net-(U12-Pad8)
- U6 pad 2: /d_bus_08 -> /reg_08
- U6 pad 3: /d_bus_09 -> /reg_09
- U6 pad 4: /d_bus_10 -> /reg_10
- U6 pad 5: /d_bus_11 -> /reg_11
- U6 pad 6: /d_bus_12 -> /reg_12
- U6 pad 7: /d_bus_13 -> /reg_13
- U6 pad 8: /d_bus_14 -> /reg_14
- U6 pad 9: /d_bus_15 -> /reg_15
- U7 pad 1: GND -> +5V
- U7 pad 11: /reg_07 -> /a_bus_07
- U7 pad 12: /reg_06 -> /a_bus_06
- U7 pad 13: /reg_05 -> /a_bus_05
- U7 pad 14: /reg_04 -> /a_bus_04
- U7 pad 15: /reg_03 -> /a_bus_03
- U7 pad 16: /reg_02 -> /a_bus_02
- U7 pad 17: /reg_01 -> /a_bus_01
- U7 pad 18: /reg_00 -> /a_bus_00
- U7 pad 19: /~x_bus_write -> Net-(U12-Pad6)
- U7 pad 2: /x_bus_00 -> /reg_00
- U7 pad 3: /x_bus_01 -> /reg_01
- U7 pad 4: /x_bus_02 -> /reg_02
- U7 pad 5: /x_bus_03 -> /reg_03
- U7 pad 6: /x_bus_04 -> /reg_04
- U7 pad 7: /x_bus_05 -> /reg_05
- U7 pad 8: /x_bus_06 -> /reg_06
- U7 pad 9: /x_bus_07 -> /reg_07
- U8 pad 1: GND -> +5V
- U8 pad 11: /reg_07 -> /a_bus_15
- U8 pad 12: /reg_14 -> /a_bus_14
- U8 pad 13: /reg_13 -> /a_bus_13
- U8 pad 14: /reg_12 -> /a_bus_12
- U8 pad 15: /reg_11 -> /a_bus_11
- U8 pad 16: /reg_10 -> /a_bus_10
- U8 pad 17: /reg_09 -> /a_bus_09
- U8 pad 18: /reg_08 -> /a_bus_08
- U8 pad 19: /~x_bus_write -> Net-(U12-Pad6)
- U8 pad 2: /x_bus_08 -> /reg_08
- U8 pad 3: /x_bus_09 -> /reg_09
- U8 pad 4: /x_bus_10 -> /reg_10
- U8 pad 5: /x_bus_11 -> /reg_11
- U8 pad 6: /x_bus_12 -> /reg_12
- U8 pad 7: /x_bus_13 -> /reg_13
- U8 pad 8: /x_bus_14 -> /reg_14
- U8 pad 9: /x_bus_15 -> /reg_15
- U9 pad 19: /~y_bus_write -> /DBG
- U9 pad 2: /y_bus_00 -> Net-(D1-Pad2)
- U9 pad 3: /y_bus_01 -> Net-(D2-Pad2)
- U9 pad 4: /y_bus_02 -> Net-(D3-Pad2)
- U9 pad 5: /y_bus_03 -> Net-(D4-Pad2)
- U9 pad 6: /y_bus_04 -> Net-(D5-Pad2)
- U9 pad 7: /y_bus_05 -> Net-(D6-Pad2)
- U9 pad 8: /y_bus_06 -> Net-(D7-Pad2)
- U9 pad 9: /y_bus_07 -> Net-(D8-Pad2)
Other:
- board outline removed
- board text removed: "DaisyX"
- board text removed: "General Purpose Register"
- board text removed: "© 2020 Chad Rempp"

Commit message: Completed GPR 1.2 PCB and started lots of other things. * Started ALU * Updated Constant Reg * Completed v1.2 GPR * Added random symbols * Updated Memory * Updated plots
Parts:
- removed J2: Interconnect B, Connector_PinHeader_2.54mm:PinHeader_2x17_P2.54mm_Horizontal
- J1: value Interconnect A -> Interconnect; footprint Connector_PinHeader_2.54mm:PinHeader_2x17_P2.54mm_Horizontal -> Connector_PCBEdge:BUS_PCI
- moved D22 233.7 mm to (-52.0, 71.9)
- moved R5 217.9 mm to (-29.7, 8.37), turned to 90 degrees
- moved D17 215.8 mm to (-40.0, 71.9)
- moved R9 213.7 mm to (-21.5, 43.8)
- moved D18 209.8 mm to (-34.0, 71.9)
- moved R19 207.6 mm to (-6.87, 10.9)
- moved D9 203.8 mm to (-28.0, 68.5)
- moved D15 201.1 mm to (-52.0, 68.5)
- moved R17 200.9 mm to (-12.3, 43.5)
- moved R18 200.9 mm to (-8.00, 43.5)
- moved R22 200.7 mm to (-21.6, 40.4)
- moved R2 200.3 mm to (-10.8, 28.3)
- moved R12 199.3 mm to (-10.8, 23.2)
- moved R10 198.7 mm to (-10.7, 53.6)
- moved D20 195.8 mm to (-22.0, 71.9)
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Connections:
- net Net-(U12-Pad6) renamed /~a_bus_write_CLK
- net Net-(U12-Pad8) renamed /~d_bus_write_CLK
- D1 pad 1: Net-(D1-Pad1) -> GND
- D10 pad 1: Net-(D10-Pad1) -> GND
- D11 pad 1: Net-(D11-Pad1) -> GND
- D12 pad 1: Net-(D12-Pad1) -> GND
- D13 pad 1: Net-(D13-Pad1) -> GND
- D14 pad 1: Net-(D14-Pad1) -> GND
- D15 pad 1: Net-(D15-Pad1) -> GND
- D16 pad 1: Net-(D16-Pad1) -> GND
- D17 pad 1: Net-(D17-Pad1) -> GND
- D18 pad 1: Net-(D18-Pad1) -> GND
- D19 pad 1: Net-(D19-Pad1) -> GND
- D2 pad 1: Net-(D2-Pad1) -> GND
- D20 pad 1: Net-(D20-Pad1) -> GND
- D21 pad 1: Net-(D21-Pad1) -> GND
- D22 pad 1: Net-(D22-Pad1) -> GND
- D23 pad 1: Net-(D23-Pad1) -> GND
- D3 pad 1: Net-(D3-Pad1) -> GND
- D4 pad 1: Net-(D4-Pad1) -> GND
- D5 pad 1: Net-(D5-Pad1) -> GND
- D6 pad 1: Net-(D6-Pad1) -> GND
- D7 pad 1: Net-(D7-Pad1) -> GND
- D8 pad 1: Net-(D8-Pad1) -> GND
- D9 pad 1: Net-(D9-Pad1) -> GND
- R1 pad 1: Net-(D1-Pad1) -> Net-(R1-Pad1)
- R1 pad 2: GND -> Net-(D1-Pad2)
- R10 pad 1: Net-(D10-Pad1) -> Net-(R10-Pad1)
- R10 pad 2: GND -> Net-(D10-Pad2)
- R11 pad 1: Net-(D11-Pad1) -> Net-(R11-Pad1)
- R11 pad 2: GND -> Net-(D11-Pad2)
- R12 pad 1: Net-(D12-Pad1) -> Net-(R12-Pad1)
- R12 pad 2: GND -> Net-(D12-Pad2)
- R13 pad 1: Net-(D13-Pad1) -> Net-(R13-Pad1)
- R13 pad 2: GND -> Net-(D13-Pad2)
- R14 pad 1: Net-(D14-Pad1) -> Net-(R14-Pad1)
- R14 pad 2: GND -> Net-(D14-Pad2)
- R15 pad 1: Net-(D15-Pad1) -> Net-(R15-Pad1)
- R15 pad 2: GND -> Net-(D15-Pad2)
- R16 pad 1: Net-(D16-Pad1) -> Net-(R16-Pad1)
- R16 pad 2: GND -> Net-(D16-Pad2)
- R17 pad 1: Net-(D17-Pad1) -> Net-(R17-Pad1)
- R17 pad 2: Net-(R17-Pad2) -> Net-(D17-Pad2)
- R18 pad 1: Net-(D18-Pad1) -> Net-(R18-Pad1)
- R18 pad 2: Net-(R17-Pad2) -> Net-(D18-Pad2)
- R19 pad 1: Net-(D19-Pad1) -> Net-(R19-Pad1)
- R19 pad 2: Net-(R17-Pad2) -> Net-(D19-Pad2)
- R2 pad 1: Net-(D2-Pad1) -> Net-(R2-Pad1)
- R2 pad 2: GND -> Net-(D2-Pad2)
- R20 pad 1: Net-(D20-Pad1) -> Net-(R20-Pad1)
- R20 pad 2: Net-(R17-Pad2) -> Net-(D20-Pad2)
- R21 pad 1: Net-(D21-Pad1) -> Net-(R21-Pad1)
- R21 pad 2: Net-(R17-Pad2) -> Net-(D21-Pad2)
- R22 pad 1: Net-(D22-Pad1) -> Net-(R22-Pad1)
- R22 pad 2: Net-(R17-Pad2) -> Net-(D22-Pad2)
- R23 pad 1: Net-(D23-Pad1) -> Net-(R23-Pad1)
- R23 pad 2: Net-(R17-Pad2) -> Net-(D23-Pad2)
- R3 pad 1: Net-(D3-Pad1) -> Net-(R3-Pad1)
- R3 pad 2: GND -> Net-(D3-Pad2)
- R4 pad 1: Net-(D4-Pad1) -> Net-(R4-Pad1)
- R4 pad 2: GND -> Net-(D4-Pad2)
- R5 pad 1: Net-(D5-Pad1) -> Net-(R5-Pad1)
- R5 pad 2: GND -> Net-(D5-Pad2)
- R6 pad 1: Net-(D6-Pad1) -> Net-(R6-Pad1)
- R6 pad 2: GND -> Net-(D6-Pad2)
- R7 pad 1: Net-(D7-Pad1) -> Net-(R7-Pad1)
- R7 pad 2: GND -> Net-(D7-Pad2)
- R8 pad 1: Net-(D8-Pad1) -> Net-(R8-Pad1)
- R8 pad 2: GND -> Net-(D8-Pad2)
- R9 pad 1: Net-(D9-Pad1) -> Net-(R9-Pad1)
- R9 pad 2: GND -> Net-(D9-Pad2)
- U1 pad 11: /d_bus_read -> /~d_bus_read
- U1 pad 14: /~RST -> /RST
- U10 pad 19: /DBG -> /~DBG
- U10 pad 2: Net-(D9-Pad2) -> Net-(R9-Pad1)
- U10 pad 3: Net-(D10-Pad2) -> Net-(R10-Pad1)
- U10 pad 4: Net-(D11-Pad2) -> Net-(R11-Pad1)
- U10 pad 5: Net-(D12-Pad2) -> Net-(R12-Pad1)
- U10 pad 6: Net-(D13-Pad2) -> Net-(R13-Pad1)
- U10 pad 7: Net-(D14-Pad2) -> Net-(R14-Pad1)
- U10 pad 8: Net-(D15-Pad2) -> Net-(R15-Pad1)
- U10 pad 9: Net-(D16-Pad2) -> Net-(R16-Pad1)
- U11 pad 19: /DBG -> /~DBG
- U11 pad 2: Net-(D17-Pad2) -> Net-(R17-Pad1)
- U11 pad 3: Net-(D18-Pad2) -> Net-(R18-Pad1)
- U11 pad 4: Net-(D19-Pad2) -> Net-(R19-Pad1)
- U11 pad 5: Net-(D20-Pad2) -> Net-(R20-Pad1)
- U11 pad 6: Net-(D21-Pad2) -> Net-(R21-Pad1)
- U11 pad 7: Net-(D22-Pad2) -> Net-(R22-Pad1)
- U11 pad 8: Net-(D23-Pad2) -> Net-(R23-Pad1)
- U12 pad 1: /RST -> /d_bus_read
- U12 pad 2: /RST -> /d_bus_read
- U12 pad 3: /~RST -> /~d_bus_read
- U2 pad 11: /d_bus_read -> /~d_bus_read
- U2 pad 14: /~RST -> /RST
- U3 pad 11: /d_bus_read -> /~d_bus_read
- U3 pad 14: /~RST -> /RST
- U4 pad 11: /d_bus_read -> /~d_bus_read
- U4 pad 14: /~RST -> /RST
- U9 pad 19: /DBG -> /~DBG
- U9 pad 2: Net-(D1-Pad2) -> Net-(R1-Pad1)
- U9 pad 3: Net-(D2-Pad2) -> Net-(R2-Pad1)
- U9 pad 4: Net-(D3-Pad2) -> Net-(R3-Pad1)
- U9 pad 5: Net-(D4-Pad2) -> Net-(R4-Pad1)
- U9 pad 6: Net-(D5-Pad2) -> Net-(R5-Pad1)
- U9 pad 7: Net-(D6-Pad2) -> Net-(R6-Pad1)
- U9 pad 8: Net-(D7-Pad2) -> Net-(R7-Pad1)
- U9 pad 9: Net-(D8-Pad2) -> Net-(R8-Pad1)
