File: cpu/Timer/TimerModule.kicad_pcb (KiCad board)
At the start: 2 copper layers, 90.6 x 58.6 mm, 17 parts, among them J1 Interconnect, U1 LM555, U2 74LS00, U3 74LS00, U4 74LS365

Commit message: Upgrade to KiCad 6 and commit a bunch of random stuff
Parts:
- D1: value ~CLK -> ~{CLK}
Connections:
- net ~CLK renamed ~{CLK}
Other:
- net class Default removed
