File: cpu/ConstantRegister/ConstantRegisterModule.sch (KiCad schematic (older format))
At the start: 76 parts

Commit message: Completed GPR 1.2 PCB and started lots of other things. * Started ALU * Updated Constant Reg * Completed v1.2 GPR * Added random symbols * Updated Memory * Updated plots
Connections:
- net labels added: md_bus_00
- net labels removed: mem_bus_00
Changed lines of the file:
@@
 $EndComp
 Text Label 1500 5200 1    50   ~ 0
-mem_bus_00
+md_bus_00
 $EndSCHEMATC
