File: cpu/Memory/MemoryModule.sch (KiCad schematic (older format))
At the start: 0 parts

Commit message: Completed GPR 1.2 PCB and started lots of other things. * Started ALU * Updated Constant Reg * Completed v1.2 GPR * Added random symbols * Updated Memory * Updated plots
Parts:
- added C1, C10, C11, C12, C13, C14, C15, C16, C2, C3, C4, C5, C6, C7, C8, C9: C, symbol Device:C
- added D1, D10, D11, D12, D13, D14, D15, D16, D17, D18, D19, D2, D20, D21, D22, D23, D24, D25, D26, D27, D28, D29, D3, D30, D31, D32, D4, D5, D6, D7, D8, D9: LED_ALT, symbol Device:LED_ALT
- added J1: Interconnect, symbol cpu_custom_symbols:Bus_PCI_32bit_5V
- added R1, R10, R11, R12, R13, R14, R15, R16, R17, R18, R19, R2, R20, R21, R22, R23, R24, R25, R26, R27, R28, R29, R3, R30, R31, R32, R4, R5, R6, R7, R8, R9: 220R, symbol Device:R
- added U1, U2, U3, U4: AT28C64B-15PU, DIP1555W45P254L3733H482Q28, symbol AT28C64B-15PU:AT28C64B-15PU
- added U10: 74LS139, symbol 74xx:74LS139
- added U11: 74LS08, symbol 74xx:74LS08
- added U12, U13, U14, U15: 74LS245, symbol 74xx:74LS245
- added U5, U6, U7, U8: AS6C62256, symbol KaiBader:AS6C62256
- added U9: 74LS173, symbol 74xx:74LS173
Connections:
- net labels added: +5V, BANK, GND, MEMRQ, RAM1_CE, RAM2_CE, RD, ROM1_CE, ROM2_CE, RST, WR, a_bus_00, a_bus_01, a_bus_02, a_bus_03, a_bus_04, a_bus_05, a_bus_06, a_bus_07, a_bus_08, a_bus_09, a_bus_10, a_bus_11, a_bus_12, a_bus_13, a_bus_14, a_bus_15, md_bus_00, md_bus_01, md_bus_02, md_bus_03, md_bus_04, md_bus_05, md_bus_06, md_bus_07, md_bus_08, md_bus_09, md_bus_10, md_bus_11, md_bus_12, md_bus_13, md_bus_14, md_bus_15, ram_13, ram_14, ~DBG
- wire segments 0 -> 588
- no-connect marks 0 -> 91
Other:
- note added: "RAM 1A"
- note added: "RAM 1B"
- note added: "RAM 2A"
- note added: "RAM 2B"
- note added: "ROM 1A"
- note added: "ROM 1B"
- note added: "ROM 2A"
- note added: "ROM 2B"
- note added: "a_bus [0,12]"
- note added: "mem_data [0,7]"
- note added: "mem_data [8,15]"
