File: cpu/Memory/MemoryModule.sch (KiCad schematic (older format))
At the start: 96 parts, among them J1 Interconnect, U1 AT28C64B-15PU, U10 74LS139, U11 74LS08, U12 74LS245, U13 74LS245, U14 74LS245, U15 74LS245, U2 AT28C64B-15PU, U3 AT28C64B-15PU, U4 AT28C64B-15PU, U5 AS6C62256, U6 AS6C62256, U7 AS6C62256, U8 AS6C62256, U9 74LS173

Commit message: Upgrade to KiCad 6 and commit a bunch of random stuff
Parts:
- added C17: C, symbol Device:C
- added U16: 74LS08, symbol 74xx:74LS08
Connections:
- wire segments 588 -> 610
Other:
- moved on the sheet: U11A, U11B
Changed lines of the file:
@@
 $Comp
 L 74xx:74LS08 U11
-U 1 1 5FA2101C
-P 2550 850
-F 0 "U11" H 2550 1050 50  0000 C CNN
-F 1 "74LS08" H 2550 650 50  0000 C CNN
-F 2 "" H 2550 850 50  0001 C CNN
-F 3 "http://www.ti.com/lit/gpn/sn74LS08" H 2550 850 50  0001 C CNN
-	1    2550 850
-	1    0    0    -1
-$EndComp
-$Comp
-L 74xx:74LS08 U11
-U 2 1 5FA22C43
-P 2550 1400
-F 0 "U11" H 2550 1600 50  0000 C CNN
-F 1 "74LS08" H 2550 1200 50  0000 C CNN
-F 2 "" H 2550 1400 50  0001 C CNN
-F 3 "http://www.ti.com/lit/gpn/sn74LS08" H 2550 1400 50  0001 C CNN
-	2    2550 1400
-	1    0    0    -1
-$EndComp
-$Comp
-L 74xx:74LS08 U11
 U 3 1 5FA24593
 P 5500 7750
@@
 Wire Wire Line
 	7350 700  7350 1250
-NoConn ~ 2850 850
-NoConn ~ 2250 750
-NoConn ~ 2250 950
-NoConn ~ 2250 1300
-NoConn ~ 2250 1500
-NoConn ~ 2850 1400
 NoConn ~ 1050 850
 NoConn ~ 1050 950
@@
 	12150 6250 4250 6250
 Wire Wire Line
-	7500 9200 7600 9100
-Wire Wire Line
-	7500 7450 7400 7350
+	8100 6600 8000 6500
 Wire Wire Line
-	7600 7450 7500 7350
+	8650 6600 8550 6500
 Wire Wire Line
-	7300 7450 7200 7350
+	6900 6600 6800 6500
 Wire Wire Line
-	7400 7450 7300 7350
-Text Label 7600 8800 3    50   ~ 0
+	7500 6600 7400 6500
+Text Label 8050 8150 3    50   ~ 0
 MEMRQ
-Wire Wire Line
-	7600 9100 7600 8800
-Text Label 7600 7450 3    50   ~ 0
+Text Label 8650 6600 3    50   ~ 0
 RAM2_CE
 Wire Wire Line
-	7600 7800 7600 7450
-Text Label 7500 7450 3    50   ~ 0
+	8650 6950 8650 6600
+Text Label 8100 6600 3    50   ~ 0
 RAM1_CE
 Wire Wire Line
-	7500 7800 7500 7450
-Text Label 7400 7450 3    50   ~ 0
+	8100 6950 8100 6600
+Text Label 7500 6600 3    50   ~ 0
 ROM2_CE
 Wire Wire Line
-	7400 7800 7400 7450
-Text Label 7300 7450 3    50   ~ 0
+	7500 6950 7500 6600
+Text Label 6900 6600 3    50   ~ 0
 ROM1_CE
 Wire Wire Line
-	7300 7800 7300 7450
+	6900 6950 6900 6600
 Text Label 7300 8800 3    50   ~ 0
 a_bus_15
@@
 $EndComp
 Connection ~ 1550 4800
+Wire Wire Line
+	7300 7800 7300 7700
+Wire Wire Line
+	7300 7700 6800 7700
+Wire Wire Line
+	6800 7700 6800 7550
+$Comp
+L power:GND #PWR021
+U 1 1 621EA472
+P 7600 8900
+F 0 "#PWR021" H 7600 8650 50  0001 C CNN
+F 1 "GND" H 7605 8727 50  0000 C CNN
+F 2 "" H 7600 8900 50  0001 C CNN
+F 3 "" H 7600 8900 50  0001 C CNN
+	1    7600 8900
+	1    0    0    -1
+$EndComp
+Wire Wire Line
+	7600 8800 7600 8900
+$Comp
+L 74xx:74LS08 U11
+U 2 1 5FA22C43
+P 7500 7250
+F 0 "U11" H 7500 7450 50  0000 C CNN
+F 1 "74LS08" H 7500 7050 50  0000 C CNN
+F 2 "" H 7500 7250 50  0001 C CNN
+F 3 "http://www.ti.com/lit/gpn/sn74LS08" H 7500 7250 50  0001 C CNN
+	2    7500 7250
+	0    -1   -1   0
+$EndComp
+$Comp
+L 74xx:74LS08 U11
+U 1 1 5FA2101C
+P 6900 7250
+F 0 "U11" H 6900 7450 50  0000 C CNN
+F 1 "74LS08" H 6900 7050 50  0000 C CNN
+F 2 "" H 6900 7250 50  0001 C CNN
+F 3 "http://www.ti.com/lit/gpn/sn74LS08" H 6900 7250 50  0001 C CNN
+	1    6900 7250
+	0    -1   -1   0
+$EndComp
+Wire Wire Line
+	7400 7550 7400 7800
+Wire Wire Line
+	7000 7550 7000 7650
+Wire Wire Line
+	8050 7650 8050 8450
+Wire Wire Line
+	7600 7550 7600 7650
+Wire Wire Line
+	7000 7650 7600 7650
+Connection ~ 7600 7650
+Wire Wire Line
+	7600 7650 8050 7650
+$Comp
+L 74xx:74LS08 U16
+U 1 1 61F530B4
+P 8100 7250
+F 0 "U16" H 8150 7450 50  0000 R CNN
+F 1 "74LS08" H 8250 7050 50  0000 R CNN
+F 2 "" H 8100 7250 50  0001 C CNN
+F 3 "http://www.ti.com/lit/gpn/sn74LS08" H 8100 7250 50  0001 C CNN
+	1    8100 7250
+	0    -1   -1   0
+$EndComp
+$Comp
+L 74xx:74LS08 U16
+U 2 1 61F59A9B
+P 8650 7250
+F 0 "U16" H 8700 7450 50  0000 R CNN
+F 1 "74LS08" H 8800 7050 50  0000 R CNN
+F 2 "" H 8650 7250 50  0001 C CNN
+F 3 "http://www.ti.com/lit/gpn/sn74LS08" H 8650 7250 50  0001 C CNN
+	2    8650 7250
+	0    -1   -1   0
+$EndComp
+$Comp
+L 74xx:74LS08 U16
+U 3 1 61F5E633
+P 2850 1100
+F 0 "U16" H 2850 1425 50  0000 C CNN
+F 1 "74LS08" H 2850 1334 50  0000 C CNN
+F 2 "" H 2850 1100 50  0001 C CNN
+F 3 "http://www.ti.com/lit/gpn/sn74LS08" H 2850 1100 50  0001 C CNN
+	3    2850 1100
+	1    0    0    -1
+$EndComp
+$Comp
+L 74xx:74LS08 U16
+U 4 1 61F61DD9
+P 2850 1700
+F 0 "U16" H 2850 2025 50  0000 C CNN
+F 1 "74LS08" H 2850 1934 50  0000 C CNN
+F 2 "" H 2850 1700 50  0001 C CNN
+F 3 "http://www.ti.com/lit/gpn/sn74LS08" H 2850 1700 50  0001 C CNN
+	4    2850 1700
+	1    0    0    -1
+$EndComp
+$Comp
+L 74xx:74LS08 U16
+U 5 1 61F6613F
+P 8600 9850
+F 0 "U16" H 8650 10200 50  0000 L CNN
+F 1 "74LS08" H 8450 9850 50  0000 L CNN
+F 2 "" H 8600 9850 50  0001 C CNN
+F 3 "http://www.ti.com/lit/gpn/sn74LS08" H 8600 9850 50  0001 C CNN
+	5    8600 9850
+	1    0    0    -1
+$EndComp
+Wire Wire Line
+	8050 7650 8200 7650
+Wire Wire Line
+	8200 7650 8200 7550
+Connection ~ 8050 7650
+Wire Wire Line
+	8200 7650 8750 7650
+Wire Wire Line
+	8750 7650 8750 7550
+Connection ~ 8200 7650
+Wire Wire Line
+	8550 7750 8550 7550
+Wire Wire Line
+	7500 7800 7500 7700
+Wire Wire Line
+	7500 7700 8000 7700
+Wire Wire Line
+	8000 7700 8000 7550
+Wire Wire Line
+	7600 7800 7600 7750
+Wire Wire Line
+	7600 7750 8550 7750
+Wire Wire Line
+	8600 9350 9100 9350
+Connection ~ 9100 9350
+Wire Wire Line
+	8600 10350 9100 10350
+Connection ~ 9100 10350
+$Comp
+L Device:C C17
+U 1 1 6238C9E5
+P 11850 10050
+F 0 "C17" H 11850 10150 50  0000 L CNN
+F 1 "C" H 11850 9950 50  0000 L CNN
+F 2 "" H 11888 9900 50  0001 C CNN
+F 3 "~" H 11850 10050 50  0001 C CNN
+	1    11850 10050
+	1    0    0    -1
+$EndComp
+Wire Wire Line
+	11650 9900 11850 9900
+Connection ~ 11650 9900
+Wire Wire Line
+	11650 10200 11850 10200
+Connection ~ 11650 10200
+NoConn ~ 3150 1100
+NoConn ~ 2550 1000
+NoConn ~ 2550 1200
+NoConn ~ 2550 1600
+NoConn ~ 2550 1800
+NoConn ~ 3150 1700
 $EndSCHEMATC
