File: cpu/Memory/MemoryModule.kicad_pcb (KiCad board)
At the start: 2 copper layers, 0 parts

Commit message: Started memory pcb layout
Parts:
- added C1: 1uf, Capacitor_SMD:C_0603_1608Metric_Pad1.08x0.95mm_HandSolder, F.Cu at (78.2, 90.7)
- added C10: 1uf, Capacitor_SMD:C_0603_1608Metric_Pad1.08x0.95mm_HandSolder, F.Cu at (203.7, 87.6)
- added C11: 1uf, Capacitor_SMD:C_0603_1608Metric_Pad1.08x0.95mm_HandSolder, F.Cu at (188.5, 110.5)
- added C12: 1uf, Capacitor_SMD:C_0603_1608Metric_Pad1.08x0.95mm_HandSolder, F.Cu at (203.7, 110.5)
- added C13: 1uf, Capacitor_SMD:C_0603_1608Metric_Pad1.08x0.95mm_HandSolder, F.Cu at (221.5, 87.6)
- added C14: 1uf, Capacitor_SMD:C_0603_1608Metric_Pad1.08x0.95mm_HandSolder, F.Cu at (236.7, 87.6)
- added C15: 1uf, Capacitor_SMD:C_0603_1608Metric_Pad1.08x0.95mm_HandSolder, F.Cu at (221.5, 110.5)
- added C16: 1uf, Capacitor_SMD:C_0603_1608Metric_Pad1.08x0.95mm_HandSolder, F.Cu at (236.7, 110.5)
- added C17: 1uf, Capacitor_SMD:C_0603_1608Metric_Pad1.08x0.95mm_HandSolder, F.Cu at (157.5, 64.3)
- added C18: 1uf, Capacitor_SMD:C_0603_1608Metric_Pad1.08x0.95mm_HandSolder, F.Cu at (169.9, 64.3)
- added C19: 1uf, Capacitor_SMD:C_0603_1608Metric_Pad1.08x0.95mm_HandSolder, F.Cu at (182.4, 64.3)
- added C2: 1uf, Capacitor_SMD:C_0603_1608Metric_Pad1.08x0.95mm_HandSolder, F.Cu at (98.6, 90.7)
- added C20: 1uf, Capacitor_SMD:C_0603_1608Metric_Pad1.08x0.95mm_HandSolder, F.Cu at (227.1, 64.8)
- added C21: 1uf, Capacitor_SMD:C_0603_1608Metric_Pad1.08x0.95mm_HandSolder, F.Cu at (193.5, 64.8)
- added C22: 1uf, Capacitor_SMD:C_0603_1608Metric_Pad1.08x0.95mm_HandSolder, F.Cu at (204.7, 64.8)
- added C23: 1uf, Capacitor_SMD:C_0603_1608Metric_Pad1.08x0.95mm_HandSolder, F.Cu at (215.9, 64.8)
- added C24: 1uf, Capacitor_SMD:C_0603_1608Metric_Pad1.08x0.95mm_HandSolder, F.Cu at (90.9, 87.1)
- added C25: 1uf, Capacitor_SMD:C_0603_1608Metric_Pad1.08x0.95mm_HandSolder, F.Cu at (70.6, 87.1)
- added C26: 1uf, Capacitor_SMD:C_0603_1608Metric_Pad1.08x0.95mm_HandSolder, F.Cu at (137.7, 87.1)
- added C27: 1uf, Capacitor_SMD:C_0603_1608Metric_Pad1.08x0.95mm_HandSolder, F.Cu at (117.3, 87.1)
- added C3: 1uf, Capacitor_SMD:C_0603_1608Metric_Pad1.08x0.95mm_HandSolder, F.Cu at (118.9, 90.7)
- added C4: 1uf, Capacitor_SMD:C_0603_1608Metric_Pad1.08x0.95mm_HandSolder, F.Cu at (139.2, 90.7)
- added C41: 10uf, Capacitor_SMD:CP_Elec_4x5.4, F.Cu at (97.0, 84.6)
- added C42: 10uf, Capacitor_SMD:CP_Elec_4x5.4, F.Cu at (163.1, 84.6)
- added C43: 10uf, Capacitor_SMD:CP_Elec_4x5.4, F.Cu at (196.1, 84.6)
- added C44: 10uf, Capacitor_SMD:CP_Elec_4x5.4, F.Cu at (229.1, 84.6)
- added C5: 1uf, Capacitor_SMD:C_0603_1608Metric_Pad1.08x0.95mm_HandSolder, F.Cu at (155.4, 87.6)
- added C6: 1uf, Capacitor_SMD:C_0603_1608Metric_Pad1.08x0.95mm_HandSolder, F.Cu at (170.7, 87.6)
- added C7: 1uf, Capacitor_SMD:C_0603_1608Metric_Pad1.08x0.95mm_HandSolder, F.Cu at (155.4, 110.5)
- added C8: 1uf, Capacitor_SMD:C_0603_1608Metric_Pad1.08x0.95mm_HandSolder, F.Cu at (170.7, 110.5)
- added C9: 1uf, Capacitor_SMD:C_0603_1608Metric_Pad1.08x0.95mm_HandSolder, F.Cu at (188.5, 87.6)
- added D1: LED, LED_SMD:LED_1206_3216Metric_Pad1.42x1.75mm_HandSolder, F.Cu at (91.7, 65.5)
- added D10: LED, LED_SMD:LED_1206_3216Metric_Pad1.42x1.75mm_HandSolder, F.Cu at (68.8, 65.5)
- added D11: LED, LED_SMD:LED_1206_3216Metric_Pad1.42x1.75mm_HandSolder, F.Cu at (66.3, 65.5)
- added D12: LED, LED_SMD:LED_1206_3216Metric_Pad1.42x1.75mm_HandSolder, F.Cu at (63.8, 65.5)
- added D13: LED, LED_SMD:LED_1206_3216Metric_Pad1.42x1.75mm_HandSolder, F.Cu at (61.2, 65.5)
- added D14: LED, LED_SMD:LED_1206_3216Metric_Pad1.42x1.75mm_HandSolder, F.Cu at (58.7, 65.5)
- added D15: LED, LED_SMD:LED_1206_3216Metric_Pad1.42x1.75mm_HandSolder, F.Cu at (56.1, 65.5)
- added D16: LED, LED_SMD:LED_1206_3216Metric_Pad1.42x1.75mm_HandSolder, F.Cu at (53.6, 65.5)
- added D17: LED, LED_SMD:LED_1206_3216Metric_Pad1.42x1.75mm_HandSolder, F.Cu at (138.7, 65.5)
- added D18: LED, LED_SMD:LED_1206_3216Metric_Pad1.42x1.75mm_HandSolder, F.Cu at (136.1, 65.5)
- added D19: LED, LED_SMD:LED_1206_3216Metric_Pad1.42x1.75mm_HandSolder, F.Cu at (133.6, 65.5)
- added D2: LED, LED_SMD:LED_1206_3216Metric_Pad1.42x1.75mm_HandSolder, F.Cu at (89.2, 65.5)
- added D20: LED, LED_SMD:LED_1206_3216Metric_Pad1.42x1.75mm_HandSolder, F.Cu at (131.1, 65.5)
- added D21: LED, LED_SMD:LED_1206_3216Metric_Pad1.42x1.75mm_HandSolder, F.Cu at (128.5, 65.5)
- added D22: LED, LED_SMD:LED_1206_3216Metric_Pad1.42x1.75mm_HandSolder, F.Cu at (126.0, 65.5)
- added D23: LED, LED_SMD:LED_1206_3216Metric_Pad1.42x1.75mm_HandSolder, F.Cu at (123.4, 65.5)
- added D24: LED, LED_SMD:LED_1206_3216Metric_Pad1.42x1.75mm_HandSolder, F.Cu at (120.9, 65.5)
- added D25: LED, LED_SMD:LED_1206_3216Metric_Pad1.42x1.75mm_HandSolder, F.Cu at (118.4, 65.5)
- added D26: LED, LED_SMD:LED_1206_3216Metric_Pad1.42x1.75mm_HandSolder, F.Cu at (115.8, 65.5)
- added D27: LED, LED_SMD:LED_1206_3216Metric_Pad1.42x1.75mm_HandSolder, F.Cu at (113.3, 65.5)
- added D28: LED, LED_SMD:LED_1206_3216Metric_Pad1.42x1.75mm_HandSolder, F.Cu at (110.7, 65.5)
- added D29: LED, LED_SMD:LED_1206_3216Metric_Pad1.42x1.75mm_HandSolder, F.Cu at (108.2, 65.5)
- added D3: LED, LED_SMD:LED_1206_3216Metric_Pad1.42x1.75mm_HandSolder, F.Cu at (86.6, 65.5)
- added D30: LED, LED_SMD:LED_1206_3216Metric_Pad1.42x1.75mm_HandSolder, F.Cu at (105.7, 65.5)
- added D31: LED, LED_SMD:LED_1206_3216Metric_Pad1.42x1.75mm_HandSolder, F.Cu at (103.1, 65.5)
- added D32: LED, LED_SMD:LED_1206_3216Metric_Pad1.42x1.75mm_HandSolder, F.Cu at (100.6, 65.5)
- added D4: LED, LED_SMD:LED_1206_3216Metric_Pad1.42x1.75mm_HandSolder, F.Cu at (84.1, 65.5)
- added D5: LED, LED_SMD:LED_1206_3216Metric_Pad1.42x1.75mm_HandSolder, F.Cu at (81.5, 65.5)
- added D6: LED, LED_SMD:LED_1206_3216Metric_Pad1.42x1.75mm_HandSolder, F.Cu at (79.0, 65.5)
- added D7: LED, LED_SMD:LED_1206_3216Metric_Pad1.42x1.75mm_HandSolder, F.Cu at (76.5, 65.5)
- added D8: LED, LED_SMD:LED_1206_3216Metric_Pad1.42x1.75mm_HandSolder, F.Cu at (73.9, 65.5)
- added D9: LED, LED_SMD:LED_1206_3216Metric_Pad1.42x1.75mm_HandSolder, F.Cu at (71.4, 65.5)
- added J1: Interconnect, Connector_PCBEdge:BUS_PCI, F.Cu at (197.5, 138.5)
- added J2: Expansion Connector A, Connector_PinHeader_1.27mm:PinHeader_1x24_P1.27mm_Vertical, F.Cu at (52.3, 96.0)
- added J3: Expansion Connector B, Connector_PinHeader_1.27mm:PinHeader_1x24_P1.27mm_Vertical, F.Cu at (245.4, 96.0)
- added REF**: OSHW-Logo2_7.3x6mm_SilkScreen, Symbol:OSHW-Logo2_7.3x6mm_SilkScreen, F.Cu at (232.9, 70.4)
- added RN1: 220R, Resistor_SMD:R_Array_Convex_8x0602, F.Cu at (82.8, 74.4)
- added RN2: 220R, Resistor_SMD:R_Array_Convex_8x0602, F.Cu at (62.5, 74.4)
- added RN3: 220R, Resistor_SMD:R_Array_Convex_8x0602, F.Cu at (129.8, 74.4)
- added RN4: 220R, Resistor_SMD:R_Array_Convex_8x0602, F.Cu at (109.5, 74.4)
- added U1: AT28C64B-15PU, Package_DIP:DIP-28_W15.24mm, F.Cu at (63.8, 93.5)
- added U10: AS6C6264-55PCN, Package_SO:SOIC-28W_7.5x18.7mm_P1.27mm, F.Cu at (199.6, 98.6)
- added U11: AS6C6264-55PCN, Package_SO:SOIC-28W_7.5x18.7mm_P1.27mm, F.Cu at (184.4, 121.4)
- added U12: AS6C6264-55PCN, Package_SO:SOIC-28W_7.5x18.7mm_P1.27mm, F.Cu at (199.6, 121.4)
- added U13: AS6C6264-55PCN, Package_SO:SOIC-28W_7.5x18.7mm_P1.27mm, F.Cu at (217.4, 98.6)
- added U14: AS6C6264-55PCN, Package_SO:SOIC-28W_7.5x18.7mm_P1.27mm, F.Cu at (232.7, 98.6)
- added U15: AS6C6264-55PCN, Package_SO:SOIC-28W_7.5x18.7mm_P1.27mm, F.Cu at (217.4, 121.4)
- added U16: AS6C6264-55PCN, Package_SO:SOIC-28W_7.5x18.7mm_P1.27mm, F.Cu at (232.7, 121.4)
- added U17: 74LS173, Package_SO:SOIC-16_3.9x9.9mm_P1.27mm, F.Cu at (155.4, 71.9)
- added U18: 74LS139, Package_SO:SOIC-16_3.9x9.9mm_P1.27mm, F.Cu at (168.1, 71.9)
- added U19: 74LS139, Package_SO:SOIC-16_3.9x9.9mm_P1.27mm, F.Cu at (180.3, 71.9)
- added U2: AT28C64B-15PU, Package_DIP:DIP-28_W15.24mm, F.Cu at (84.1, 93.5)
- added U20: 74LS04, Package_SO:SOIC-14_3.9x8.7mm_P1.27mm, F.Cu at (225.0, 71.9)
- added U21: 74LS08, Package_SO:SOIC-14_3.9x8.7mm_P1.27mm, F.Cu at (191.5, 71.9)
- added U22: 74LS08, Package_SO:SOIC-14_3.9x8.7mm_P1.27mm, F.Cu at (202.7, 71.9)
- added U23: 74LS08, Package_SO:SOIC-14_3.9x8.7mm_P1.27mm, F.Cu at (213.9, 71.9)
- added U24: 74LS245, Package_SO:SOIC-20W_7.5x12.8mm_P1.27mm, F.Cu at (82.8, 83.3)
- added U25: 74LS245, Package_SO:SOIC-20W_7.5x12.8mm_P1.27mm, F.Cu at (62.5, 83.3)
- added U26: 74LS245, Package_SO:SOIC-20W_7.5x12.8mm_P1.27mm, F.Cu at (129.8, 83.3)
- added U27: 74LS245, Package_SO:SOIC-20W_7.5x12.8mm_P1.27mm, F.Cu at (109.5, 83.3)
- added U3: AT28C64B-15PU, Package_DIP:DIP-28_W15.24mm, F.Cu at (104.4, 93.5)
- added U4: AT28C64B-15PU, Package_DIP:DIP-28_W15.24mm, F.Cu at (124.7, 93.5)
- added U5: AS6C6264-55PCN, Package_SO:SOIC-28W_7.5x18.7mm_P1.27mm, F.Cu at (151.4, 98.6)
- added U6: AS6C6264-55PCN, Package_SO:SOIC-28W_7.5x18.7mm_P1.27mm, F.Cu at (166.6, 98.6)
- added U7: AS6C6264-55PCN, Package_SO:SOIC-28W_7.5x18.7mm_P1.27mm, F.Cu at (151.4, 121.4)
- added U8: AS6C6264-55PCN, Package_SO:SOIC-28W_7.5x18.7mm_P1.27mm, F.Cu at (166.6, 121.4)
- added U9: AS6C6264-55PCN, Package_SO:SOIC-28W_7.5x18.7mm_P1.27mm, F.Cu at (184.4, 98.6)
Routing:
- net +5V: track 0.00 -> 659.5 mm, vias 0 -> 19
- net /a_bus_00: track 0.00 -> 409.1 mm, vias 0 -> 14
- net /a_bus_01: track 0.00 -> 391.7 mm, vias 0 -> 15
- net /a_bus_02: track 0.00 -> 389.3 mm, vias 0 -> 14
- net /a_bus_04: track 0.00 -> 388.2 mm, vias 0 -> 14
- net /a_bus_12: track 0.00 -> 387.4 mm, vias 0 -> 14
- net /a_bus_03: track 0.00 -> 386.3 mm, vias 0 -> 14
- net /a_bus_08: track 0.00 -> 378.3 mm, vias 0 -> 12
- net /a_bus_05: track 0.00 -> 373.9 mm, vias 0 -> 14
- net /a_bus_06: track 0.00 -> 371.8 mm, vias 0 -> 14
- net /a_bus_07: track 0.00 -> 367.6 mm, vias 0 -> 14
- net /md_bus_15: track 0.00 -> 366.7 mm, vias 0 -> 11
- net /md_bus_14: track 0.00 -> 361.0 mm, vias 0 -> 10
- net /a_bus_10: track 0.00 -> 359.7 mm, vias 0 -> 13
- net /md_bus_08: track 0.00 -> 358.2 mm, vias 0 -> 12
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Other:
- board outline added: 197.8 x 80 mm
- board text added: "Base Memory Module"
- board text added: "CPU u16"
- board text added: "© 2022 Chad Rempp"
