File: cpu/Memory/MemoryModule.kicad_sch (KiCad schematic)
At the start: 98 parts, among them J1 Interconnect, U1 AT28C64B-15PU, U10 74LS139, U11 74LS08, U12 74LS245, U13 74LS245, U14 74LS245, U15 74LS245, U16 74LS08, U2 AT28C64B-15PU, U3 AT28C64B-15PU, U4 AT28C64B-15PU, U5 AS6C62256, U6 AS6C62256, U7 AS6C62256, U8 AS6C62256, U9 74LS173

Commit message: Memory module v2.0 schematic
Parts:
- removed D1, D10, D11, D12, D13, D14, D15, D16, D17, D18, D19, D2, D20, D21, D22, D23, D24, D25, D26, D27, D28, D29, D3, D30, D31, D32, D4, D5, D6, D7, D8, D9: LED_ALT, symbol Device:LED_ALT
- removed U1, U2, U3, U4: AT28C64B-15PU, DIP1555W45P254L3733H482Q28, symbol AT28C64B-15PU:AT28C64B-15PU
- removed U10: 74LS139, symbol 74xx:74LS139
- removed U11, U16: 74LS08, symbol 74xx:74LS08
- removed U5, U6, U7, U8: AS6C62256, symbol KaiBader:AS6C62256
- removed U9: 74LS173, symbol 74xx:74LS173
- added C18, C19, C20, C21, C22, C23, C24, C25, C26, C27, C28, C29, C30, C31, C32, C33, C34, C35, C36, C37, C38, C39, C40, C45, C46, C47, C48, C49, C50, C51, C52, C53, C54, C55, C56, C57, C58, C59, C60, C61, C62, C63, C64, C65, C66, C67, C68: C, symbol Device:C
- added C41, C42, C43, C44: 10uf, symbol Device:C_Polarized_US
- added D1, D10, D11, D12, D13, D14, D15, D16, D17, D18, D19, D2, D20, D21, D22, D23, D24, D25, D26, D27, D28, D29, D3, D30, D31, D32, D4, D5, D6, D7, D8, D9: LED, symbol Device:LED
- added J2: Expansion Connector A, symbol Connector:Conn_01x24_Female
- added J3: Expansion Connector B, symbol Connector:Conn_01x24_Female
- added U1, U31, U32: 74LS138, symbol 74xx:74LS138
- added U10, U11, U16, U17, U2, U21, U22, U23, U24, U25, U26, U27, U28, U3, U33, U34, U35, U36, U37, U38, U39, U4, U40, U41, U42, U43, U44, U45, U46, U47, U48, U49, U5, U50, U51, U52, U53, U54, U55, U56, U57, U58, U59, U60, U61, U62, U63, U64: CY7C128A-45PC, Maxim-DS1220AD-200+-*, symbol Maxim_DS1220AD:DS1220AD-200+
- added U18, U6: 74LS139, symbol 74xx:74LS139
- added U19, U20, U29, U30: AT28C64B-15PU, DIP1555W45P254L3733H482Q28, symbol AT28C64B-15PU.lib:AT28C64B-15PU
- added U7: 74LS08, symbol 74xx:74LS08
- added U8: 74LS173, symbol 74xx:74LS173
- added U9: 74LS04, symbol 74xx:74LS04
Connections:
- net +5V: now also C18.1, C19.1, C20.1, C21.1, C22.1, C23.1, C24.1, C25.1, C26.1, C27.1, C28.1, C29.1, C30.1, C31.1, C32.1, C33.1, C34.1, C35.1, C36.1, C37.1, C38.1, C39.1, C40.1, C41.1, C42.1, C43.1, C44.1, C45.1, C46.1, C47.1, C48.1, C49.1, C50.1, C51.1, C52.1, C53.1, C54.1, C55.1, C56.1, C57.1, C58.1, C59.1, C60.1, C61.1, C62.1, C63.1, C64.1, C65.1, C66.1, C67.1, C68.1, J2.2 (Pin_2), J3.2 (Pin_2), J3.3 (Pin_3), U1.16 (VCC), U1.6 (E3), U10.24 (VCC), U11.24 (VCC), U16.24 (VCC), U17.24 (VCC), U18.16 (VCC), U19.28 (VCC), U2.24 (VCC), U20.28 (VCC), U21.24 (VCC), U22.24 (VCC), U23.24 (VCC), U24.24 (VCC), U25.24 (VCC), U26.24 (VCC), U27.24 (VCC), U28.24 (VCC), U29.28 (VCC), U3.24 (VCC), U30.28 (VCC), U31.16 (VCC), U31.6 (E3), U32.16 (VCC), U32.6 (E3), U33.24 (VCC), U34.24 (VCC), U35.24 (VCC), U36.24 (VCC), U37.24 (VCC), U38.24 (VCC), U39.24 (VCC), U4.24 (VCC), U40.24 (VCC), U41.24 (VCC), U42.24 (VCC), U43.24 (VCC), U44.24 (VCC), U45.24 (VCC), U46.24 (VCC), U47.24 (VCC), U48.24 (VCC), U49.24 (VCC), U5.24 (VCC), U50.24 (VCC), U51.24 (VCC), U52.24 (VCC), U53.24 (VCC), U54.24 (VCC), U55.24 (VCC), U56.24 (VCC), U57.24 (VCC), U58.24 (VCC), U59.24 (VCC), U6.16 (VCC), U60.24 (VCC), U61.24 (VCC), U62.24 (VCC), U63.24 (VCC), U64.24 (VCC), U7.14 (VCC), U8.10 (E2), U8.16 (VCC), U8.9 (E1), U9.14 (VCC)
- net BANK: now also U8.7 (Cp)
- net GND: now also C18.2, C19.2, C20.2, C21.2, C22.2, C23.2, C24.2, C25.2, C26.2, C27.2, C28.2, C29.2, C30.2, C31.2, C32.2, C33.2, C34.2, C35.2, C36.2, C37.2, C38.2, C39.2, C40.2, C41.2, C42.2, C43.2, C44.2, C45.2, C46.2, C47.2, C48.2, C49.2, C50.2, C51.2, C52.2, C53.2, C54.2, C55.2, C56.2, C57.2, C58.2, C59.2, C60.2, C61.2, C62.2, C63.2, C64.2, C65.2, C66.2, C67.2, C68.2, D1.1 (K), D10.1 (K), D11.1 (K), D12.1 (K), D13.1 (K), D14.1 (K), D15.1 (K), D16.1 (K), D17.1 (K), D18.1 (K), D19.1 (K), D2.1 (K), D20.1 (K), D21.1 (K), D22.1 (K), D23.1 (K), D24.1 (K), D25.1 (K), D26.1 (K), D27.1 (K), D28.1 (K), D29.1 (K), D3.1 (K), D30.1 (K), D31.1 (K), D32.1 (K), D4.1 (K), D5.1 (K), D6.1 (K), D7.1 (K), D8.1 (K), D9.1 (K), J2.1 (Pin_1), J3.1 (Pin_1), U1.8 (GND), U10.12 (GND), U11.12 (GND), U16.12 (GND), U17.12 (GND), U18.8 (GND), U19.14 (GND), U2.12 (GND), U20.14 (GND), U21.12 (GND), U22.12 (GND), U23.12 (GND), U24.12 (GND), U25.12 (GND), U26.12 (GND), U27.12 (GND), U28.12 (GND), U29.14 (GND), U3.12 (GND), U30.14 (GND), U31.8 (GND), U32.8 (GND), U33.12 (GND), U34.12 (GND), U35.12 (GND), U36.12 (GND), U37.12 (GND), U38.12 (GND), U39.12 (GND), U4.12 (GND), U40.12 (GND), U41.12 (GND), U42.12 (GND), U43.12 (GND), U44.12 (GND), U45.12 (GND), U46.12 (GND), U47.12 (GND), U48.12 (GND), U49.12 (GND), U5.12 (GND), U50.12 (GND), U51.12 (GND), U52.12 (GND), U53.12 (GND), U54.12 (GND), U55.12 (GND), U56.12 (GND), U57.12 (GND), U58.12 (GND), U59.12 (GND), U6.1 (E), U6.15 (E), U6.8 (GND), U60.12 (GND), U61.12 (GND), U62.12 (GND), U63.12 (GND), U64.12 (GND), U7.7 (GND), U8.1 (Oe1), U8.2 (Oe2), U8.8 (GND), U9.7 (GND)
- net MEMRQ: now also U18.1 (E)
- net RD: now also U10.20 (~{OE}), U11.20 (~{OE}), U16.20 (~{OE}), U17.20 (~{OE}), U19.22 (~{OE}), U2.20 (~{OE}), U20.22 (~{OE}), U21.20 (~{OE}), U22.20 (~{OE}), U23.20 (~{OE}), U24.20 (~{OE}), U25.20 (~{OE}), U26.20 (~{OE}), U27.20 (~{OE}), U28.20 (~{OE}), U29.22 (~{OE}), U3.20 (~{OE}), U30.22 (~{OE}), U33.20 (~{OE}), U34.20 (~{OE}), U35.20 (~{OE}), U36.20 (~{OE}), U37.20 (~{OE}), U38.20 (~{OE}), U39.20 (~{OE}), U4.20 (~{OE}), U40.20 (~{OE}), U41.20 (~{OE}), U42.20 (~{OE}), U43.20 (~{OE}), U44.20 (~{OE}), U45.20 (~{OE}), U46.20 (~{OE}), U47.20 (~{OE}), U48.20 (~{OE}), U49.20 (~{OE}), U5.20 (~{OE}), U50.20 (~{OE}), U51.20 (~{OE}), U52.20 (~{OE}), U53.20 (~{OE}), U54.20 (~{OE}), U55.20 (~{OE}), U56.20 (~{OE}), U57.20 (~{OE}), U58.20 (~{OE}), U59.20 (~{OE}), U60.20 (~{OE}), U61.20 (~{OE}), U62.20 (~{OE}), U63.20 (~{OE}), U64.20 (~{OE})
- net RST: now also U8.15 (Mr)
- net WR: now also U10.21 (~{WE}), U11.21 (~{WE}), U16.21 (~{WE}), U17.21 (~{WE}), U19.27 (~{WE}), U2.21 (~{WE}), U20.27 (~{WE}), U21.21 (~{WE}), U22.21 (~{WE}), U23.21 (~{WE}), U24.21 (~{WE}), U25.21 (~{WE}), U26.21 (~{WE}), U27.21 (~{WE}), U28.21 (~{WE}), U29.27 (~{WE}), U3.21 (~{WE}), U30.27 (~{WE}), U33.21 (~{WE}), U34.21 (~{WE}), U35.21 (~{WE}), U36.21 (~{WE}), U37.21 (~{WE}), U38.21 (~{WE}), U39.21 (~{WE}), U4.21 (~{WE}), U40.21 (~{WE}), U41.21 (~{WE}), U42.21 (~{WE}), U43.21 (~{WE}), U44.21 (~{WE}), U45.21 (~{WE}), U46.21 (~{WE}), U47.21 (~{WE}), U48.21 (~{WE}), U49.21 (~{WE}), U5.21 (~{WE}), U50.21 (~{WE}), U51.21 (~{WE}), U52.21 (~{WE}), U53.21 (~{WE}), U54.21 (~{WE}), U55.21 (~{WE}), U56.21 (~{WE}), U57.21 (~{WE}), U58.21 (~{WE}), U59.21 (~{WE}), U60.21 (~{WE}), U61.21 (~{WE}), U62.21 (~{WE}), U63.21 (~{WE}), U64.21 (~{WE})
- net a_bus_00: now also J2.24 (Pin_24), U10.8 (A0), U11.8 (A0), U16.8 (A0), U17.8 (A0), U19.10 (A0), U2.8 (A0), U20.10 (A0), U21.8 (A0), U22.8 (A0), U23.8 (A0), U24.8 (A0), U25.8 (A0), U26.8 (A0), U27.8 (A0), U28.8 (A0), U29.10 (A0), U3.8 (A0), U30.10 (A0), U33.8 (A0), U34.8 (A0), U35.8 (A0), U36.8 (A0), U37.8 (A0), U38.8 (A0), U39.8 (A0), U4.8 (A0), U40.8 (A0), U41.8 (A0), U42.8 (A0), U43.8 (A0), U44.8 (A0), U45.8 (A0), U46.8 (A0), U47.8 (A0), U48.8 (A0), U49.8 (A0), U5.8 (A0), U50.8 (A0), U51.8 (A0), U52.8 (A0), U53.8 (A0), U54.8 (A0), U55.8 (A0), U56.8 (A0), U57.8 (A0), U58.8 (A0), U59.8 (A0), U60.8 (A0), U61.8 (A0), U62.8 (A0), U63.8 (A0), U64.8 (A0)
- net a_bus_01: now also J2.23 (Pin_23), U10.7 (A1), U11.7 (A1), U16.7 (A1), U17.7 (A1), U19.9 (A1), U2.7 (A1), U20.9 (A1), U21.7 (A1), U22.7 (A1), U23.7 (A1), U24.7 (A1), U25.7 (A1), U26.7 (A1), U27.7 (A1), U28.7 (A1), U29.9 (A1), U3.7 (A1), U30.9 (A1), U33.7 (A1), U34.7 (A1), U35.7 (A1), U36.7 (A1), U37.7 (A1), U38.7 (A1), U39.7 (A1), U4.7 (A1), U40.7 (A1), U41.7 (A1), U42.7 (A1), U43.7 (A1), U44.7 (A1), U45.7 (A1), U46.7 (A1), U47.7 (A1), U48.7 (A1), U49.7 (A1), U5.7 (A1), U50.7 (A1), U51.7 (A1), U52.7 (A1), U53.7 (A1), U54.7 (A1), U55.7 (A1), U56.7 (A1), U57.7 (A1), U58.7 (A1), U59.7 (A1), U60.7 (A1), U61.7 (A1), U62.7 (A1), U63.7 (A1), U64.7 (A1)
- net a_bus_02: now also J2.22 (Pin_22), U10.6 (A2), U11.6 (A2), U16.6 (A2), U17.6 (A2), U19.8 (A2), U2.6 (A2), U20.8 (A2), U21.6 (A2), U22.6 (A2), U23.6 (A2), U24.6 (A2), U25.6 (A2), U26.6 (A2), U27.6 (A2), U28.6 (A2), U29.8 (A2), U3.6 (A2), U30.8 (A2), U33.6 (A2), U34.6 (A2), U35.6 (A2), U36.6 (A2), U37.6 (A2), U38.6 (A2), U39.6 (A2), U4.6 (A2), U40.6 (A2), U41.6 (A2), U42.6 (A2), U43.6 (A2), U44.6 (A2), U45.6 (A2), U46.6 (A2), U47.6 (A2), U48.6 (A2), U49.6 (A2), U5.6 (A2), U50.6 (A2), U51.6 (A2), U52.6 (A2), U53.6 (A2), U54.6 (A2), U55.6 (A2), U56.6 (A2), U57.6 (A2), U58.6 (A2), U59.6 (A2), U60.6 (A2), U61.6 (A2), U62.6 (A2), U63.6 (A2), U64.6 (A2)
- net a_bus_03: now also J2.21 (Pin_21), U10.5 (A3), U11.5 (A3), U16.5 (A3), U17.5 (A3), U19.7 (A3), U2.5 (A3), U20.7 (A3), U21.5 (A3), U22.5 (A3), U23.5 (A3), U24.5 (A3), U25.5 (A3), U26.5 (A3), U27.5 (A3), U28.5 (A3), U29.7 (A3), U3.5 (A3), U30.7 (A3), U33.5 (A3), U34.5 (A3), U35.5 (A3), U36.5 (A3), U37.5 (A3), U38.5 (A3), U39.5 (A3), U4.5 (A3), U40.5 (A3), U41.5 (A3), U42.5 (A3), U43.5 (A3), U44.5 (A3), U45.5 (A3), U46.5 (A3), U47.5 (A3), U48.5 (A3), U49.5 (A3), U5.5 (A3), U50.5 (A3), U51.5 (A3), U52.5 (A3), U53.5 (A3), U54.5 (A3), U55.5 (A3), U56.5 (A3), U57.5 (A3), U58.5 (A3), U59.5 (A3), U60.5 (A3), U61.5 (A3), U62.5 (A3), U63.5 (A3), U64.5 (A3)
- net a_bus_04: now also J2.20 (Pin_20), U10.4 (A4), U11.4 (A4), U16.4 (A4), U17.4 (A4), U19.6 (A4), U2.4 (A4), U20.6 (A4), U21.4 (A4), U22.4 (A4), U23.4 (A4), U24.4 (A4), U25.4 (A4), U26.4 (A4), U27.4 (A4), U28.4 (A4), U29.6 (A4), U3.4 (A4), U30.6 (A4), U33.4 (A4), U34.4 (A4), U35.4 (A4), U36.4 (A4), U37.4 (A4), U38.4 (A4), U39.4 (A4), U4.4 (A4), U40.4 (A4), U41.4 (A4), U42.4 (A4), U43.4 (A4), U44.4 (A4), U45.4 (A4), U46.4 (A4), U47.4 (A4), U48.4 (A4), U49.4 (A4), U5.4 (A4), U50.4 (A4), U51.4 (A4), U52.4 (A4), U53.4 (A4), U54.4 (A4), U55.4 (A4), U56.4 (A4), U57.4 (A4), U58.4 (A4), U59.4 (A4), U60.4 (A4), U61.4 (A4), U62.4 (A4), U63.4 (A4), U64.4 (A4)
- net a_bus_05: now also J2.19 (Pin_19), U10.3 (A5), U11.3 (A5), U16.3 (A5), U17.3 (A5), U19.5 (A5), U2.3 (A5), U20.5 (A5), U21.3 (A5), U22.3 (A5), U23.3 (A5), U24.3 (A5), U25.3 (A5), U26.3 (A5), U27.3 (A5), U28.3 (A5), U29.5 (A5), U3.3 (A5), U30.5 (A5), U33.3 (A5), U34.3 (A5), U35.3 (A5), U36.3 (A5), U37.3 (A5), U38.3 (A5), U39.3 (A5), U4.3 (A5), U40.3 (A5), U41.3 (A5), U42.3 (A5), U43.3 (A5), U44.3 (A5), U45.3 (A5), U46.3 (A5), U47.3 (A5), U48.3 (A5), U49.3 (A5), U5.3 (A5), U50.3 (A5), U51.3 (A5), U52.3 (A5), U53.3 (A5), U54.3 (A5), U55.3 (A5), U56.3 (A5), U57.3 (A5), U58.3 (A5), U59.3 (A5), U60.3 (A5), U61.3 (A5), U62.3 (A5), U63.3 (A5), U64.3 (A5)
- net a_bus_06: now also J2.18 (Pin_18), U10.2 (A6), U11.2 (A6), U16.2 (A6), U17.2 (A6), U19.4 (A6), U2.2 (A6), U20.4 (A6), U21.2 (A6), U22.2 (A6), U23.2 (A6), U24.2 (A6), U25.2 (A6), U26.2 (A6), U27.2 (A6), U28.2 (A6), U29.4 (A6), U3.2 (A6), U30.4 (A6), U33.2 (A6), U34.2 (A6), U35.2 (A6), U36.2 (A6), U37.2 (A6), U38.2 (A6), U39.2 (A6), U4.2 (A6), U40.2 (A6), U41.2 (A6), U42.2 (A6), U43.2 (A6), U44.2 (A6), U45.2 (A6), U46.2 (A6), U47.2 (A6), U48.2 (A6), U49.2 (A6), U5.2 (A6), U50.2 (A6), U51.2 (A6), U52.2 (A6), U53.2 (A6), U54.2 (A6), U55.2 (A6), U56.2 (A6), U57.2 (A6), U58.2 (A6), U59.2 (A6), U60.2 (A6), U61.2 (A6), U62.2 (A6), U63.2 (A6), U64.2 (A6)
- net a_bus_07: now also J2.17 (Pin_17), U10.1 (A7), U11.1 (A7), U16.1 (A7), U17.1 (A7), U19.3 (A7), U2.1 (A7), U20.3 (A7), U21.1 (A7), U22.1 (A7), U23.1 (A7), U24.1 (A7), U25.1 (A7), U26.1 (A7), U27.1 (A7), U28.1 (A7), U29.3 (A7), U3.1 (A7), U30.3 (A7), U33.1 (A7), U34.1 (A7), U35.1 (A7), U36.1 (A7), U37.1 (A7), U38.1 (A7), U39.1 (A7), U4.1 (A7), U40.1 (A7), U41.1 (A7), U42.1 (A7), U43.1 (A7), U44.1 (A7), U45.1 (A7), U46.1 (A7), U47.1 (A7), U48.1 (A7), U49.1 (A7), U5.1 (A7), U50.1 (A7), U51.1 (A7), U52.1 (A7), U53.1 (A7), U54.1 (A7), U55.1 (A7), U56.1 (A7), U57.1 (A7), U58.1 (A7), U59.1 (A7), U60.1 (A7), U61.1 (A7), U62.1 (A7), U63.1 (A7), U64.1 (A7)
- net a_bus_08: now also J2.16 (Pin_16), U10.23 (A8), U11.23 (A8), U16.23 (A8), U17.23 (A8), U19.25 (A8), U2.23 (A8), U20.25 (A8), U21.23 (A8), U22.23 (A8), U23.23 (A8), U24.23 (A8), U25.23 (A8), U26.23 (A8), U27.23 (A8), U28.23 (A8), U29.25 (A8), U3.23 (A8), U30.25 (A8), U33.23 (A8), U34.23 (A8), U35.23 (A8), U36.23 (A8), U37.23 (A8), U38.23 (A8), U39.23 (A8), U4.23 (A8), U40.23 (A8), U41.23 (A8), U42.23 (A8), U43.23 (A8), U44.23 (A8), U45.23 (A8), U46.23 (A8), U47.23 (A8), U48.23 (A8), U49.23 (A8), U5.23 (A8), U50.23 (A8), U51.23 (A8), U52.23 (A8), U53.23 (A8), U54.23 (A8), U55.23 (A8), U56.23 (A8), U57.23 (A8), U58.23 (A8), U59.23 (A8), U60.23 (A8), U61.23 (A8), U62.23 (A8), U63.23 (A8), U64.23 (A8)
- net a_bus_09: now also J2.15 (Pin_15), U10.22 (A9), U11.22 (A9), U16.22 (A9), U17.22 (A9), U19.24 (A9), U2.22 (A9), U20.24 (A9), U21.22 (A9), U22.22 (A9), U23.22 (A9), U24.22 (A9), U25.22 (A9), U26.22 (A9), U27.22 (A9), U28.22 (A9), U29.24 (A9), U3.22 (A9), U30.24 (A9), U33.22 (A9), U34.22 (A9), U35.22 (A9), U36.22 (A9), U37.22 (A9), U38.22 (A9), U39.22 (A9), U4.22 (A9), U40.22 (A9), U41.22 (A9), U42.22 (A9), U43.22 (A9), U44.22 (A9), U45.22 (A9), U46.22 (A9), U47.22 (A9), U48.22 (A9), U49.22 (A9), U5.22 (A9), U50.22 (A9), U51.22 (A9), U52.22 (A9), U53.22 (A9), U54.22 (A9), U55.22 (A9), U56.22 (A9), U57.22 (A9), U58.22 (A9), U59.22 (A9), U60.22 (A9), U61.22 (A9), U62.22 (A9), U63.22 (A9), U64.22 (A9)
- net a_bus_10: now also J2.14 (Pin_14), U10.19 (A10), U11.19 (A10), U16.19 (A10), U17.19 (A10), U19.21 (A10), U2.19 (A10), U20.21 (A10), U21.19 (A10), U22.19 (A10), U23.19 (A10), U24.19 (A10), U25.19 (A10), U26.19 (A10), U27.19 (A10), U28.19 (A10), U29.21 (A10), U3.19 (A10), U30.21 (A10), U33.19 (A10), U34.19 (A10), U35.19 (A10), U36.19 (A10), U37.19 (A10), U38.19 (A10), U39.19 (A10), U4.19 (A10), U40.19 (A10), U41.19 (A10), U42.19 (A10), U43.19 (A10), U44.19 (A10), U45.19 (A10), U46.19 (A10), U47.19 (A10), U48.19 (A10), U49.19 (A10), U5.19 (A10), U50.19 (A10), U51.19 (A10), U52.19 (A10), U53.19 (A10), U54.19 (A10), U55.19 (A10), U56.19 (A10), U57.19 (A10), U58.19 (A10), U59.19 (A10), U60.19 (A10), U61.19 (A10), U62.19 (A10), U63.19 (A10), U64.19 (A10)
- net a_bus_11: now also J2.13 (Pin_13), U1.1 (A0), U19.23 (A11), U20.23 (A11), U29.23 (A11), U30.23 (A11), U31.1 (A0), U32.1 (A0)
- net a_bus_12: now also J2.12 (Pin_12), U1.2 (A1), U19.2 (A12), U20.2 (A12), U29.2 (A12), U30.2 (A12), U31.2 (A1), U32.2 (A1)
- net a_bus_13: now also J2.11 (Pin_11), U1.3 (A2), U31.3 (A2), U32.3 (A2), U7.5, U9.1
- net a_bus_14: now also J2.10 (Pin_10), U18.2 (A0)
- net a_bus_15: now also J2.9 (Pin_9), U18.3 (A1)
- net md_bus_00: now also U19.11 (I/O0), U2.9 (DQ0), U21.9 (DQ0), U22.9 (DQ0), U23.9 (DQ0), U24.9 (DQ0), U29.11 (I/O0), U3.9 (DQ0), U33.9 (DQ0), U34.9 (DQ0), U35.9 (DQ0), U36.9 (DQ0), U37.9 (DQ0), U38.9 (DQ0), U39.9 (DQ0), U4.9 (DQ0), U40.9 (DQ0), U49.9 (DQ0), U5.9 (DQ0), U50.9 (DQ0), U51.9 (DQ0), U52.9 (DQ0), U53.9 (DQ0), U54.9 (DQ0), U55.9 (DQ0), U56.9 (DQ0), U8.14 (D0)
- net md_bus_01: now also J3.24 (Pin_24), U19.12 (I/O1), U2.10 (DQ1), U21.10 (DQ1), U22.10 (DQ1), U23.10 (DQ1), U24.10 (DQ1), U29.12 (I/O1), U3.10 (DQ1), U33.10 (DQ1), U34.10 (DQ1), U35.10 (DQ1), U36.10 (DQ1), U37.10 (DQ1), U38.10 (DQ1), U39.10 (DQ1), U4.10 (DQ1), U40.10 (DQ1), U49.10 (DQ1), U5.10 (DQ1), U50.10 (DQ1), U51.10 (DQ1), U52.10 (DQ1), U53.10 (DQ1), U54.10 (DQ1), U55.10 (DQ1), U56.10 (DQ1), U8.13 (D1)
- net md_bus_02: now also J3.23 (Pin_23), U19.13 (I/O2), U2.11 (DQ2), U21.11 (DQ2), U22.11 (DQ2), U23.11 (DQ2), U24.11 (DQ2), U29.13 (I/O2), U3.11 (DQ2), U33.11 (DQ2), U34.11 (DQ2), U35.11 (DQ2), U36.11 (DQ2), U37.11 (DQ2), U38.11 (DQ2), U39.11 (DQ2), U4.11 (DQ2), U40.11 (DQ2), U49.11 (DQ2), U5.11 (DQ2), U50.11 (DQ2), U51.11 (DQ2), U52.11 (DQ2), U53.11 (DQ2), U54.11 (DQ2), U55.11 (DQ2), U56.11 (DQ2), U8.12 (D2)
- net md_bus_03: now also J3.22 (Pin_22), U19.15 (I/O3), U2.13 (DQ3), U21.13 (DQ3), U22.13 (DQ3), U23.13 (DQ3), U24.13 (DQ3), U29.15 (I/O3), U3.13 (DQ3), U33.13 (DQ3), U34.13 (DQ3), U35.13 (DQ3), U36.13 (DQ3), U37.13 (DQ3), U38.13 (DQ3), U39.13 (DQ3), U4.13 (DQ3), U40.13 (DQ3), U49.13 (DQ3), U5.13 (DQ3), U50.13 (DQ3), U51.13 (DQ3), U52.13 (DQ3), U53.13 (DQ3), U54.13 (DQ3), U55.13 (DQ3), U56.13 (DQ3), U8.11 (D3)
- net md_bus_04: now also J3.21 (Pin_21), U19.16 (I/O4), U2.14 (DQ4), U21.14 (DQ4), U22.14 (DQ4), U23.14 (DQ4), U24.14 (DQ4), U29.16 (I/O4), U3.14 (DQ4), U33.14 (DQ4), U34.14 (DQ4), U35.14 (DQ4), U36.14 (DQ4), U37.14 (DQ4), U38.14 (DQ4), U39.14 (DQ4), U4.14 (DQ4), U40.14 (DQ4), U49.14 (DQ4), U5.14 (DQ4), U50.14 (DQ4), U51.14 (DQ4), U52.14 (DQ4), U53.14 (DQ4), U54.14 (DQ4), U55.14 (DQ4), U56.14 (DQ4)
- net md_bus_05: now also J3.20 (Pin_20), U19.17 (I/O5), U2.15 (DQ5), U21.15 (DQ5), U22.15 (DQ5), U23.15 (DQ5), U24.15 (DQ5), U29.17 (I/O5), U3.15 (DQ5), U33.15 (DQ5), U34.15 (DQ5), U35.15 (DQ5), U36.15 (DQ5), U37.15 (DQ5), U38.15 (DQ5), U39.15 (DQ5), U4.15 (DQ5), U40.15 (DQ5), U49.15 (DQ5), U5.15 (DQ5), U50.15 (DQ5), U51.15 (DQ5), U52.15 (DQ5), U53.15 (DQ5), U54.15 (DQ5), U55.15 (DQ5), U56.15 (DQ5)
- net md_bus_06: now also J3.19 (Pin_19), U19.18 (I/O6), U2.16 (DQ6), U21.16 (DQ6), U22.16 (DQ6), U23.16 (DQ6), U24.16 (DQ6), U29.18 (I/O6), U3.16 (DQ6), U33.16 (DQ6), U34.16 (DQ6), U35.16 (DQ6), U36.16 (DQ6), U37.16 (DQ6), U38.16 (DQ6), U39.16 (DQ6), U4.16 (DQ6), U40.16 (DQ6), U49.16 (DQ6), U5.16 (DQ6), U50.16 (DQ6), U51.16 (DQ6), U52.16 (DQ6), U53.16 (DQ6), U54.16 (DQ6), U55.16 (DQ6), U56.16 (DQ6)
- net md_bus_07: now also J3.18 (Pin_18), U19.19 (I/O7), U2.17 (DQ7), U21.17 (DQ7), U22.17 (DQ7), U23.17 (DQ7), U24.17 (DQ7), U29.19 (I/O7), U3.17 (DQ7), U33.17 (DQ7), U34.17 (DQ7), U35.17 (DQ7), U36.17 (DQ7), U37.17 (DQ7), U38.17 (DQ7), U39.17 (DQ7), U4.17 (DQ7), U40.17 (DQ7), U49.17 (DQ7), U5.17 (DQ7), U50.17 (DQ7), U51.17 (DQ7), U52.17 (DQ7), U53.17 (DQ7), U54.17 (DQ7), U55.17 (DQ7), U56.17 (DQ7)
- net md_bus_08: now also J3.17 (Pin_17), U10.9 (DQ0), U11.9 (DQ0), U16.9 (DQ0), U17.9 (DQ0), U20.11 (I/O0), U25.9 (DQ0), U26.9 (DQ0), U27.9 (DQ0), U28.9 (DQ0), U30.11 (I/O0), U41.9 (DQ0), U42.9 (DQ0), U43.9 (DQ0), U44.9 (DQ0), U45.9 (DQ0), U46.9 (DQ0), U47.9 (DQ0), U48.9 (DQ0), U57.9 (DQ0), U58.9 (DQ0), U59.9 (DQ0), U60.9 (DQ0), U61.9 (DQ0), U62.9 (DQ0), U63.9 (DQ0), U64.9 (DQ0)
- net md_bus_09: now also J3.16 (Pin_16), U10.10 (DQ1), U11.10 (DQ1), U16.10 (DQ1), U17.10 (DQ1), U20.12 (I/O1), U25.10 (DQ1), U26.10 (DQ1), U27.10 (DQ1), U28.10 (DQ1), U30.12 (I/O1), U41.10 (DQ1), U42.10 (DQ1), U43.10 (DQ1), U44.10 (DQ1), U45.10 (DQ1), U46.10 (DQ1), U47.10 (DQ1), U48.10 (DQ1), U57.10 (DQ1), U58.10 (DQ1), U59.10 (DQ1), U60.10 (DQ1), U61.10 (DQ1), U62.10 (DQ1), U63.10 (DQ1), U64.10 (DQ1)
- net md_bus_10: now also J3.15 (Pin_15), U10.11 (DQ2), U11.11 (DQ2), U16.11 (DQ2), U17.11 (DQ2), U20.13 (I/O2), U25.11 (DQ2), U26.11 (DQ2), U27.11 (DQ2), U28.11 (DQ2), U30.13 (I/O2), U41.11 (DQ2), U42.11 (DQ2), U43.11 (DQ2), U44.11 (DQ2), U45.11 (DQ2), U46.11 (DQ2), U47.11 (DQ2), U48.11 (DQ2), U57.11 (DQ2), U58.11 (DQ2), U59.11 (DQ2), U60.11 (DQ2), U61.11 (DQ2), U62.11 (DQ2), U63.11 (DQ2), U64.11 (DQ2)
- net md_bus_11: now also J3.14 (Pin_14), U10.13 (DQ3), U11.13 (DQ3), U16.13 (DQ3), U17.13 (DQ3), U20.15 (I/O3), U25.13 (DQ3), U26.13 (DQ3), U27.13 (DQ3), U28.13 (DQ3), U30.15 (I/O3), U41.13 (DQ3), U42.13 (DQ3), U43.13 (DQ3), U44.13 (DQ3), U45.13 (DQ3), U46.13 (DQ3), U47.13 (DQ3), U48.13 (DQ3), U57.13 (DQ3), U58.13 (DQ3), U59.13 (DQ3), U60.13 (DQ3), U61.13 (DQ3), U62.13 (DQ3), U63.13 (DQ3), U64.13 (DQ3)
- net md_bus_12: now also J3.13 (Pin_13), U10.14 (DQ4), U11.14 (DQ4), U16.14 (DQ4), U17.14 (DQ4), U20.16 (I/O4), U25.14 (DQ4), U26.14 (DQ4), U27.14 (DQ4), U28.14 (DQ4), U30.16 (I/O4), U41.14 (DQ4), U42.14 (DQ4), U43.14 (DQ4), U44.14 (DQ4), U45.14 (DQ4), U46.14 (DQ4), U47.14 (DQ4), U48.14 (DQ4), U57.14 (DQ4), U58.14 (DQ4), U59.14 (DQ4), U60.14 (DQ4), U61.14 (DQ4), U62.14 (DQ4), U63.14 (DQ4), U64.14 (DQ4)
- net md_bus_13: now also J3.12 (Pin_12), U10.15 (DQ5), U11.15 (DQ5), U16.15 (DQ5), U17.15 (DQ5), U20.17 (I/O5), U25.15 (DQ5), U26.15 (DQ5), U27.15 (DQ5), U28.15 (DQ5), U30.17 (I/O5), U41.15 (DQ5), U42.15 (DQ5), U43.15 (DQ5), U44.15 (DQ5), U45.15 (DQ5), U46.15 (DQ5), U47.15 (DQ5), U48.15 (DQ5), U57.15 (DQ5), U58.15 (DQ5), U59.15 (DQ5), U60.15 (DQ5), U61.15 (DQ5), U62.15 (DQ5), U63.15 (DQ5), U64.15 (DQ5)
- net md_bus_14: now also J3.11 (Pin_11), U10.16 (DQ6), U11.16 (DQ6), U16.16 (DQ6), U17.16 (DQ6), U20.18 (I/O6), U25.16 (DQ6), U26.16 (DQ6), U27.16 (DQ6), U28.16 (DQ6), U30.18 (I/O6), U41.16 (DQ6), U42.16 (DQ6), U43.16 (DQ6), U44.16 (DQ6), U45.16 (DQ6), U46.16 (DQ6), U47.16 (DQ6), U48.16 (DQ6), U57.16 (DQ6), U58.16 (DQ6), U59.16 (DQ6), U60.16 (DQ6), U61.16 (DQ6), U62.16 (DQ6), U63.16 (DQ6), U64.16 (DQ6)
- net md_bus_15: now also J3.10 (Pin_10), U10.17 (DQ7), U11.17 (DQ7), U16.17 (DQ7), U17.17 (DQ7), U20.19 (I/O7), U25.17 (DQ7), U26.17 (DQ7), U27.17 (DQ7), U28.17 (DQ7), U30.19 (I/O7), U41.17 (DQ7), U42.17 (DQ7), U43.17 (DQ7), U44.17 (DQ7), U45.17 (DQ7), U46.17 (DQ7), U47.17 (DQ7), U48.17 (DQ7), U57.17 (DQ7), U58.17 (DQ7), U59.17 (DQ7), U60.17 (DQ7), U61.17 (DQ7), U62.17 (DQ7), U63.17 (DQ7), U64.17 (DQ7)
- net /bank_a_select: now reaches J1.B10 (control_07)
- net /bank_a_select: now also J3.5 (Pin_5), U1.5 (E2), U18.4 (O0), U31.5 (E2), U32.5 (E2), U7.1
- net /enable_lowbank_3: now reaches J1.B11 (control_06)
- net /enable_lowbank_3: now also J2.5 (Pin_5), U6.7 (O3)
- net /enable_lowbank_2: now reaches J1.B12 (control_05)
- net /enable_lowbank_2: now also J2.6 (Pin_6), U6.6 (O2)
- net /enable_lowbank_1: now reaches J1.B13 (control_04)
- net /enable_lowbank_1: now also J2.7 (Pin_7), U6.5 (O1)
- net at R8.2: now also D8.2 (A)
- net at R7.2: now also D7.2 (A)
- net at R6.2: now also D6.2 (A)
- net at R5.2: now also D5.2 (A)
- net at R4.2: now also D4.2 (A)
- net at R3.2: now also D3.2 (A)
- net at R2.2: now also D2.2 (A)
- net at R1.2: now also D1.2 (A)
- net at R16.2: now also D16.2 (A)
- net at R15.2: now also D15.2 (A)
- net at R14.2: now also D14.2 (A)
- net at R13.2: now also D13.2 (A)
- net at R12.2: now also D12.2 (A)
- net at R11.2: now also D11.2 (A)
- net at R10.2: now also D10.2 (A)
- net at R9.2: now also D9.2 (A)
- net at R24.2: now also D24.2 (A)
- net at R23.2: now also D23.2 (A)
- net at R22.2: now also D22.2 (A)
- net at R21.2: now also D21.2 (A)
- net at R20.2: now also D20.2 (A)
- net at R19.2: now also D19.2 (A)
- net at R18.2: now also D18.2 (A)
- net at R17.2: now also D17.2 (A)
- net at R32.2: now also D32.2 (A)
- net at R31.2: now also D31.2 (A)
- net at R30.2: now also D30.2 (A)
- net at R29.2: now also D29.2 (A)
- net at R28.2: now also D28.2 (A)
- net at R27.2: now also D27.2 (A)
- net at R26.2: now also D26.2 (A)
- net at R25.2: now also D25.2 (A)
- new net: U31.12 (O3), U51.18 (~{CE}), U59.18 (~{CE})
- new net: U31.10 (O5), U50.18 (~{CE}), U58.18 (~{CE})
- new net: U31.11 (O4), U34.18 (~{CE}), U42.18 (~{CE})
- new net: U31.13 (O2), U35.18 (~{CE}), U43.18 (~{CE})
- new net: U31.14 (O1), U52.18 (~{CE}), U60.18 (~{CE})
- new net: U31.15 (O0), U36.18 (~{CE}), U44.18 (~{CE})
- new net: U31.7 (O7), U49.18 (~{CE}), U57.18 (~{CE})
- new net: U31.9 (O6), U33.18 (~{CE}), U41.18 (~{CE})
- new net: U32.15 (O0), U40.18 (~{CE}), U48.18 (~{CE})
- new net: U7.10, U9.2
- new net: U29.20 (~{CE}), U30.20 (~{CE}), U7.8
- new net: U7.3, U7.4, U7.9
- new net: U1.11 (O4), U11.18 (~{CE}), U3.18 (~{CE})
- new net: U32.9 (O6), U37.18 (~{CE}), U45.18 (~{CE})
- new net: U19.20 (~{CE}), U20.20 (~{CE}), U7.6
- new net: U32.14 (O1), U56.18 (~{CE}), U64.18 (~{CE})
- new net: U1.10 (O5), U22.18 (~{CE}), U26.18 (~{CE})
- new net: U32.12 (O3), U55.18 (~{CE}), U63.18 (~{CE})
- new net: U32.11 (O4), U38.18 (~{CE}), U46.18 (~{CE})
- new net: U1.7 (O7), U21.18 (~{CE}), U25.18 (~{CE})
- new net: U1.15 (O0), U17.18 (~{CE}), U5.18 (~{CE})
- new net: U32.7 (O7), U53.18 (~{CE}), U61.18 (~{CE})
- new net: U1.9 (O6), U10.18 (~{CE}), U2.18 (~{CE})
- new net: U6.13 (A1), U8.5 (Q2)
- new net: U6.14 (A0), U8.6 (Q3)
- new net: U32.13 (O2), U39.18 (~{CE}), U47.18 (~{CE})
- new net: U1.12 (O3), U23.18 (~{CE}), U27.18 (~{CE})
- new net: U1.13 (O2), U16.18 (~{CE}), U4.18 (~{CE})
- new net: U1.14 (O1), U24.18 (~{CE}), U28.18 (~{CE})
- new net: U6.2 (A0), U8.4 (Q1)
- new net: U6.3 (A1), U8.3 (Q0)
- new net: U32.10 (O5), U54.18 (~{CE}), U62.18 (~{CE})
- new net /bank_b_select: J3.4 (Pin_4), U18.5 (O1)
- new net /bank_c_select: J2.4 (Pin_4), U18.6 (O2)
- new net /bank_d_select: J2.3 (Pin_3), U18.7 (O3)
- new net /enable_highbank_0: J3.9 (Pin_9), U6.12 (O0)
- new net /enable_highbank_1: J3.8 (Pin_8), U6.11 (O1)
- new net /enable_highbank_2: J3.7 (Pin_7), U6.10 (O2)
- new net /enable_highbank_3: J3.6 (Pin_6), U6.9 (O3)
- new net /enable_lowbank_0: J2.8 (Pin_8), U1.4 (E1), U31.4 (E1), U32.4 (E1), U6.4 (O0), U7.2
- no-connect marks 91 -> 90
Other:
- note added: "16 Kb"
- note added: "Bank Selection Decoding"
- note added: "Bank Switching Decoding"
- note added: "RAM Bank C:0"
- note added: "RAM C:0:0H"
- note added: "RAM C:0:0L"
- note added: "RAM C:0:1H"
- note added: "RAM C:0:1L"
- note added: "RAM C:0:2H"
- note added: "RAM C:0:2L"
- note added: "RAM C:0:3H"
- note added: "RAM C:0:3L"
- note added: "RAM C:0:4H"
- note added: "RAM C:0:4L"
- note added: "RAM C:0:5H"
- note added: "RAM C:0:5L"
- note added: "RAM C:0:6H"
- note added: "RAM C:0:6L"
- note added: "RAM C:0:7H"
- note added: "RAM C:0:7L"
- note added: "ROM A:0:0H"
- note added: "ROM A:0:0L"
- note added: "ROM A:0:1H"
- note added: "ROM A:0:1L"
- note added: "ROM Bank A:0"
- note added: "The 64 Kb address space is split into four 16 Kb blocks (A, B, C, D). Blocks are further grouped into 32 Kb groups: the low block group (A & B) and high block group (C & D). Four banks are available to be selected for blocks A, C and D. Block B is static and can not be changed, that is where the stack lives. The value set in the bank register selects the banking configuration Configurations are d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"
- note added: "The top two address lines (A14, A15) select which 16 Kb bank is active. 00 - Bank A 01 - Bank B 10 - Bank C 11 - Bank D"
- note removed: "RAM 1A"
- note removed: "RAM 1B"
- note removed: "RAM 2A"
- note removed: "RAM 2B"
- note removed: "ROM 1A"
- note removed: "ROM 1B"
- note removed: "ROM 2A"
- note removed: "ROM 2B"
- note removed: "a_bus [0,12]"
- note removed: "mem_data [0,7]"
- note removed: "mem_data [8,15]"
- moved on the sheet: C1, C10, C11, C12, C13, C14, C15, C16, C2, C3, C4, C5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

Commit message: Started memory pcb layout
Parts:
- removed C28, C29, C30, C31, C32, C33, C34, C35, C36, C37, C38, C39, C40, C45, C46, C47, C48, C49, C50, C51, C52, C53, C54, C55, C56, C57, C58, C59, C60, C61, C62, C63, C64, C65, C66, C67, C68: C, symbol Device:C
- removed R1, R10, R11, R12, R13, R14, R15, R16, R17, R18, R19, R2, R20, R21, R22, R23, R24, R25, R26, R27, R28, R29, R3, R30, R31, R32, R4, R5, R6, R7, R8, R9: 220R, symbol Device:R
- removed U1, U31, U32: 74LS138, symbol 74xx:74LS138
- removed U10, U11, U16, U17, U2, U21, U22, U23, U24, U25, U26, U27, U28, U3, U33, U34, U35, U36, U37, U38, U39, U4, U40, U41, U42, U43, U44, U45, U46, U47, U48, U49, U5, U50, U51, U52, U53, U54, U55, U56, U57, U58, U59, U60, U61, U62, U63, U64: CY7C128A-45PC, Maxim-DS1220AD-200+-*, symbol Maxim_DS1220AD:DS1220AD-200+
- removed unit 4 of U7
- removed unit 2 of U9
- added RN1, RN2, RN3, RN4: 220R, Resistor_SMD:R_Array_Convex_8x0602, symbol Device:R_Pack08
- added U10, U11, U12, U13, U14, U15, U16, U5, U6, U7, U8, U9: AS6C6264-55PCN, Package_SO:SOIC-28W_7.5x18.7mm_P1.27mm, symbol AS6C6264-55PCN:AS6C6264-55PCN
- added unit 2 of U20
- added unit 4 of U21
- added U22, U23: 74LS08, Package_SO:SOIC-14_3.9x8.7mm_P1.27mm, symbol 74xx:74LS08
- C1, C10, C11, C12, C13, C14, C15, C16, C17, C18, C19, C2, C20, C21, C22, C23, C24, C25, C26, C27, C3, C4, C5, C6, C7, C8, C9: value C -> 1uf; footprint (none) -> Capacitor_SMD:C_0603_1608Metric_Pad1.08x0.95mm_HandSolder
- C41, C42, C43, C44: footprint (none) -> Capacitor_SMD:CP_Elec_4x5.4
- D1, D10, D11, D12, D13, D14, D15, D16, D17, D18, D19, D2, D20, D21, D22, D23, D24, D25, D26, D27, D28, D29, D3, D30, D31, D32, D4, D5, D6, D7, D8, D9: footprint (none) -> LED_SMD:LED_1206_3216Metric_Pad1.42x1.75mm_HandSolder
- J1: footprint (none) -> Connector_PCBEdge:BUS_PCI
- J2, J3: footprint (none) -> Connector_PinHeader_1.27mm:PinHeader_1x24_P1.27mm_Vertical
- U1: renamed from U29; footprint DIP1555W45P254L3733H482Q28 -> Package_DIP:DIP-28_W15.24mm
- U17: renamed from U8; footprint (none) -> Package_SO:SOIC-16_3.9x9.9mm_P1.27mm
- U18: renamed from U6; footprint (none) -> Package_SO:SOIC-16_3.9x9.9mm_P1.27mm
- U19: renamed from U18; footprint (none) -> Package_SO:SOIC-16_3.9x9.9mm_P1.27mm
- U2: renamed from U30; footprint DIP1555W45P254L3733H482Q28 -> Package_DIP:DIP-28_W15.24mm
- U20: renamed from U9; footprint (none) -> Package_SO:SOIC-14_3.9x8.7mm_P1.27mm
- U21: renamed from U7; footprint (none) -> Package_SO:SOIC-14_3.9x8.7mm_P1.27mm
- U24: renamed from U12; footprint (none) -> Package_SO:SOIC-20W_7.5x12.8mm_P1.27mm; Digikey (none) -> 296-1208-1-ND
- U25: renamed from U13; footprint (none) -> Package_SO:SOIC-20W_7.5x12.8mm_P1.27mm; Digikey (none) -> 296-1208-1-ND
- U26: renamed from U14; footprint (none) -> Package_SO:SOIC-20W_7.5x12.8mm_P1.27mm; Digikey (none) -> 296-1208-1-ND
- U27: renamed from U15; footprint (none) -> Package_SO:SOIC-20W_7.5x12.8mm_P1.27mm; Digikey (none) -> 296-1208-1-ND
- U3: renamed from U19; footprint DIP1555W45P254L3733H482Q28 -> Package_DIP:DIP-28_W15.24mm
- U4: renamed from U20; footprint DIP1555W45P254L3733H482Q28 -> Package_DIP:DIP-28_W15.24mm
Connections:
- net +5V: now also U10.26 (CE2), U10.28 (Vcc), U11.26 (CE2), U11.28 (Vcc), U12.26 (CE2), U12.28 (Vcc), U13.26 (CE2), U13.28 (Vcc), U14.26 (CE2), U14.28 (Vcc), U15.26 (CE2), U15.28 (Vcc), U16.26 (CE2), U16.28 (Vcc), U22.14 (VCC), U23.14 (VCC), U5.26 (CE2), U5.28 (Vcc), U6.26 (CE2), U6.28 (Vcc), U7.26 (CE2), U7.28 (Vcc), U8.26 (CE2), U8.28 (Vcc), U9.26 (CE2), U9.28 (Vcc)
- net GND: now also U10.14 (Vss), U11.14 (Vss), U12.14 (Vss), U13.14 (Vss), U14.14 (Vss), U15.14 (Vss), U16.14 (Vss), U22.7 (GND), U23.7 (GND), U5.14 (Vss), U6.14 (Vss), U7.14 (Vss), U8.14 (Vss), U9.14 (Vss)
- net RD: now also U10.22 (~{OE}), U11.22 (~{OE}), U12.22 (~{OE}), U13.22 (~{OE}), U14.22 (~{OE}), U15.22 (~{OE}), U16.22 (~{OE}), U5.22 (~{OE}), U6.22 (~{OE}), U7.22 (~{OE}), U8.22 (~{OE}), U9.22 (~{OE})
- net WR: now also U10.27 (~{WE}), U11.27 (~{WE}), U12.27 (~{WE}), U13.27 (~{WE}), U14.27 (~{WE}), U15.27 (~{WE}), U16.27 (~{WE}), U5.27 (~{WE}), U6.27 (~{WE}), U7.27 (~{WE}), U8.27 (~{WE}), U9.27 (~{WE})
- net a_bus_00: now also U10.10 (A0), U11.10 (A0), U12.10 (A0), U13.10 (A0), U14.10 (A0), U15.10 (A0), U16.10 (A0), U5.10 (A0), U6.10 (A0), U7.10 (A0), U8.10 (A0), U9.10 (A0)
- net a_bus_01: now also U10.9 (A1), U11.9 (A1), U12.9 (A1), U13.9 (A1), U14.9 (A1), U15.9 (A1), U16.9 (A1), U5.9 (A1), U6.9 (A1), U7.9 (A1), U8.9 (A1), U9.9 (A1)
- net a_bus_02: now also U10.8 (A2), U11.8 (A2), U12.8 (A2), U13.8 (A2), U14.8 (A2), U15.8 (A2), U16.8 (A2), U5.8 (A2), U6.8 (A2), U7.8 (A2), U8.8 (A2), U9.8 (A2)
- net a_bus_03: now also U10.7 (A3), U11.7 (A3), U12.7 (A3), U13.7 (A3), U14.7 (A3), U15.7 (A3), U16.7 (A3), U5.7 (A3), U6.7 (A3), U7.7 (A3), U8.7 (A3), U9.7 (A3)
- net a_bus_04: now also U10.6 (A4), U11.6 (A4), U12.6 (A4), U13.6 (A4), U14.6 (A4), U15.6 (A4), U16.6 (A4), U5.6 (A4), U6.6 (A4), U7.6 (A4), U8.6 (A4), U9.6 (A4)
- net a_bus_05: now also U10.5 (A5), U11.5 (A5), U12.5 (A5), U13.5 (A5), U14.5 (A5), U15.5 (A5), U16.5 (A5), U5.5 (A5), U6.5 (A5), U7.5 (A5), U8.5 (A5), U9.5 (A5)
- net a_bus_06: now also U10.4 (A6), U11.4 (A6), U12.4 (A6), U13.4 (A6), U14.4 (A6), U15.4 (A6), U16.4 (A6), U5.4 (A6), U6.4 (A6), U7.4 (A6), U8.4 (A6), U9.4 (A6)
- net a_bus_07: now also U10.3 (A7), U11.3 (A7), U12.3 (A7), U13.3 (A7), U14.3 (A7), U15.3 (A7), U16.3 (A7), U5.3 (A7), U6.3 (A7), U7.3 (A7), U8.3 (A7), U9.3 (A7)
- net a_bus_08: now also U10.25 (A8), U11.25 (A8), U12.25 (A8), U13.25 (A8), U14.25 (A8), U15.25 (A8), U16.25 (A8), U5.25 (A8), U6.25 (A8), U7.25 (A8), U8.25 (A8), U9.25 (A8)
- net a_bus_09: now also U10.24 (A9), U11.24 (A9), U12.24 (A9), U13.24 (A9), U14.24 (A9), U15.24 (A9), U16.24 (A9), U5.24 (A9), U6.24 (A9), U7.24 (A9), U8.24 (A9), U9.24 (A9)
- net a_bus_10: now also U10.21 (A10), U11.21 (A10), U12.21 (A10), U13.21 (A10), U14.21 (A10), U15.21 (A10), U16.21 (A10), U5.21 (A10), U6.21 (A10), U7.21 (A10), U8.21 (A10), U9.21 (A10)
- net a_bus_11: now also U10.23 (A11), U11.23 (A11), U12.23 (A11), U13.23 (A11), U14.23 (A11), U15.23 (A11), U16.23 (A11), U5.23 (A11), U6.23 (A11), U7.23 (A11), U8.23 (A11), U9.23 (A11)
- net a_bus_12: now also U10.2 (A12), U11.2 (A12), U12.2 (A12), U13.2 (A12), U14.2 (A12), U15.2 (A12), U16.2 (A12), U5.2 (A12), U6.2 (A12), U7.2 (A12), U8.2 (A12), U9.2 (A12)
- net a_bus_13: now also U20.5, U20.9, U20.3, U22.13, U22.2, U23.10
- net md_bus_00: now also U11.11 (DQ0), U13.11 (DQ0), U15.11 (DQ0), U5.11 (DQ0), U7.11 (DQ0), U9.11 (DQ0)
- net md_bus_01: now also U11.12 (DQ1), U13.12 (DQ1), U15.12 (DQ1), U5.12 (DQ1), U7.12 (DQ1), U9.12 (DQ1)
- net md_bus_02: now also U11.13 (DQ2), U13.13 (DQ2), U15.13 (DQ2), U5.13 (DQ2), U7.13 (DQ2), U9.13 (DQ2)
- net md_bus_03: now also U11.15 (DQ3), U13.15 (DQ3), U15.15 (DQ3), U5.15 (DQ3), U7.15 (DQ3), U9.15 (DQ3)
- net md_bus_04: now also U11.16 (DQ4), U13.16 (DQ4), U15.16 (DQ4), U5.16 (DQ4), U7.16 (DQ4), U9.16 (DQ4)
- net md_bus_05: now also U11.17 (DQ5), U13.17 (DQ5), U15.17 (DQ5), U5.17 (DQ5), U7.17 (DQ5), U9.17 (DQ5)
- net md_bus_06: now also U11.18 (DQ6), U13.18 (DQ6), U15.18 (DQ6), U5.18 (DQ6), U7.18 (DQ6), U9.18 (DQ6)
- net md_bus_07: now also U11.19 (DQ7), U13.19 (DQ7), U15.19 (DQ7), U5.19 (DQ7), U7.19 (DQ7), U9.19 (DQ7)
- net md_bus_08: now also U10.11 (DQ0), U12.11 (DQ0), U14.11 (DQ0), U16.11 (DQ0), U6.11 (DQ0), U8.11 (DQ0)
- net md_bus_09: now also U10.12 (DQ1), U12.12 (DQ1), U14.12 (DQ1), U16.12 (DQ1), U6.12 (DQ1), U8.12 (DQ1)
- net md_bus_10: now also U10.13 (DQ2), U12.13 (DQ2), U14.13 (DQ2), U16.13 (DQ2), U6.13 (DQ2), U8.13 (DQ2)
- net md_bus_11: now also U10.15 (DQ3), U12.15 (DQ3), U14.15 (DQ3), U16.15 (DQ3), U6.15 (DQ3), U8.15 (DQ3)
- net md_bus_12: now also U10.16 (DQ4), U12.16 (DQ4), U14.16 (DQ4), U16.16 (DQ4), U6.16 (DQ4), U8.16 (DQ4)
- net md_bus_13: now also U10.17 (DQ5), U12.17 (DQ5), U14.17 (DQ5), U16.17 (DQ5), U6.17 (DQ5), U8.17 (DQ5)
- net md_bus_14: now also U10.18 (DQ6), U12.18 (DQ6), U14.18 (DQ6), U16.18 (DQ6), U6.18 (DQ6), U8.18 (DQ6)
- net md_bus_15: now also U10.19 (DQ7), U12.19 (DQ7), U14.19 (DQ7), U16.19 (DQ7), U6.19 (DQ7), U8.19 (DQ7)
- net /bank_b_select: now also U21.12
- net /bank_c_select: now also U22.9
- net /bank_d_select: now also U23.4
- net /enable_lowbank_0: now also U21.13, U22.10, U23.5
- net at U24.2 (A0): now also RN1.16 (R1.2)
- net at U24.3 (A1): now also RN1.15 (R2.2)
- net at U24.4 (A2): now also RN1.14 (R3.2)
- net at U24.5 (A3): now also RN1.13 (R4.2)
- net at U24.6 (A4): now also RN1.12 (R5.2)
- net at U24.7 (A5): now also RN1.11 (R6.2)
- net at U24.8 (A6): now also RN1.10 (R7.2)
- net at U24.9 (A7): now also RN1.9 (R8.2)
- net at D8.2 (A): now also RN1.8 (R8.1)
- net at D7.2 (A): now also RN1.7 (R7.1)
- net at D6.2 (A): now also RN1.6 (R6.1)
- net at D5.2 (A): now also RN1.5 (R5.1)
- net at D4.2 (A): now also RN1.4 (R4.1)
- net at D3.2 (A): now also RN1.3 (R3.1)
- net at D2.2 (A): now also RN1.2 (R2.1)
- net at D1.2 (A): now also RN1.1 (R1.1)
- net at U25.9 (A7): now also RN2.9 (R8.2)
- net at D16.2 (A): now also RN2.8 (R8.1)
- net at U25.8 (A6): now also RN2.10 (R7.2)
- net at D15.2 (A): now also RN2.7 (R7.1)
- net at U25.7 (A5): now also RN2.11 (R6.2)
- net at D14.2 (A): now also RN2.6 (R6.1)
- net at U25.6 (A4): now also RN2.12 (R5.2)
- net at D13.2 (A): now also RN2.5 (R5.1)
- net at U25.5 (A3): now also RN2.13 (R4.2)
- net at D12.2 (A): now also RN2.4 (R4.1)
- net at U25.4 (A2): now also RN2.14 (R3.2)
- net at D11.2 (A): now also RN2.3 (R3.1)
- net at U25.3 (A1): now also RN2.15 (R2.2)
- net at D10.2 (A): now also RN2.2 (R2.1)
- net at U25.2 (A0): now also RN2.16 (R1.2)
- net at D9.2 (A): now also RN2.1 (R1.1)
- net at U26.2 (A0): now also RN3.16 (R1.2)
- net at U26.3 (A1): now also RN3.15 (R2.2)
- net at U26.4 (A2): now also RN3.14 (R3.2)
- net at U26.5 (A3): now also RN3.13 (R4.2)
- net at U26.6 (A4): now also RN3.12 (R5.2)
- net at U26.7 (A5): now also RN3.11 (R6.2)
- net at U26.8 (A6): now also RN3.10 (R7.2)
- net at U26.9 (A7): now also RN3.9 (R8.2)
- net at D24.2 (A): now also RN3.8 (R8.1)
- net at D23.2 (A): now also RN3.7 (R7.1)
- net at D22.2 (A): now also RN3.6 (R6.1)
- net at D21.2 (A): now also RN3.5 (R5.1)
- net at D20.2 (A): now also RN3.4 (R4.1)
- net at D19.2 (A): now also RN3.3 (R3.1)
- net at D18.2 (A): now also RN3.2 (R2.1)
- net at D17.2 (A): now also RN3.1 (R1.1)
- net at U27.9 (A7): now also RN4.9 (R8.2)
- net at D32.2 (A): now also RN4.8 (R8.1)
- net at U27.8 (A6): now also RN4.10 (R7.2)
- net at D31.2 (A): now also RN4.7 (R7.1)
- net at U27.7 (A5): now also RN4.11 (R6.2)
- net at D30.2 (A): now also RN4.6 (R6.1)
- net at U27.6 (A4): now also RN4.12 (R5.2)
- net at D29.2 (A): now also RN4.5 (R5.1)
- net at U27.5 (A3): now also RN4.13 (R4.2)
- net at D28.2 (A): now also RN4.4 (R4.1)
- net at U27.4 (A2): now also RN4.14 (R3.2)
- net at D27.2 (A): now also RN4.3 (R3.1)
- net at U27.3 (A1): now also RN4.15 (R2.2)
- net at D26.2 (A): now also RN4.2 (R2.1)
- net at U27.2 (A0): now also RN4.16 (R1.2)
- net at D25.2 (A): now also RN4.1 (R1.1)
- net at U20.6: now also U23.2
- net at U20.8: now also U23.13
- new net: U22.3, U7.20 (~{CE}), U8.20 (~{CE})
- new net: U22.6, U5.20 (~{CE}), U6.20 (~{CE})
- new net: U20.4, U22.5
- new net: U15.20 (~{CE}), U16.20 (~{CE}), U23.8
- new net: U10.20 (~{CE}), U23.3, U9.20 (~{CE})
- new net: U23.12, U23.6, U23.9
- new net: U22.12, U22.8, U23.1
- new net: U21.11, U22.1, U22.4
- new net: U13.20 (~{CE}), U14.20 (~{CE}), U23.11
- new net: U11.20 (~{CE}), U12.20 (~{CE}), U22.11
- no-connect marks 90 -> 93
Other:
- note added: "RAM B:0:0H"
- note added: "RAM B:0:0L"
- note added: "RAM B:0:1L"
- note added: "RAM Bank B:0 (16 KB)"
- note added: "RAM Bank C:0 (16 KB)"
- note added: "RAM Bank D:0 (16 KB)"
- note added: "RAM D:0:0H"
- note added: "RAM D:0:0L"
- note added: "RAM D:0:1L"
- note added: "TODO: * Validate RAM footprints are ok"
- note removed: "RAM Bank C:0"
- note removed: "RAM C:0:1H"
- note removed: "RAM C:0:2H"
- note removed: "RAM C:0:2L"
- note removed: "RAM C:0:3H"
- note removed: "RAM C:0:3L"
- note removed: "RAM C:0:4H"
- note removed: "RAM C:0:4L"
- note removed: "RAM C:0:5H"
- note removed: "RAM C:0:5L"
- note removed: "RAM C:0:6H"
- note removed: "RAM C:0:6L"
- note removed: "RAM C:0:7H"
- note removed: "RAM C:0:7L"
- moved on the sheet: C1, C10, C11, C12, C13, C14, C15, C16, C17, C18, C19, C2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

Commit message: Mem module fixes
Connections:
- net /bank_b_select: now also U22.1, U22.4; no longer U21.12
- net /enable_highbank_0: now also U22.10, U23.5
- net /enable_lowbank_0: no longer U21.13, U22.10, U23.5
- now unconnected: U21.11
- no-connect marks 93 -> 96
Other:
- note added: "Expansion Connectors"
- moved on the sheet: C1, C10, C11, C12, C13, C14, C15, C16, C17, C18, C19, C2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
