File: cpu/ALU/ALUModule.kicad_pcb (KiCad board)
At the start: 2 copper layers, 168 parts, among them J1 Interconnect 1, J2 Interconnect 2, J3 Interconnect 3, U1 74LS245, U10 74LS253, U11 74LS253, U12 74LS253, U13 74LS253, U14 74LS253, U15 74LS253, U16 74LS253, U17 74LS253, U18 74LS253, U19 74LS245, U2 74LS245, U20 74LS245, U21 74LS02, U22 74LS08, U23 74LS08, U24 74LS253, U25 74LS253, U26 74LS253, U27 74LS253, U28 74LS253, U29 74LS253, U3 74LS253, U30 74LS253, U31 74LS253, U32 74LS253, U33 74LS02, U34 74LS86, U35 74LS283, U36 74LS283, U37 74LS283, U38 74LS283, U39 74LS574, U4 74LS253, U40 74LS574, U41 74LS574, U42 74LS574, U43 74LS574, U44 74LS253, U45 74LS245, U46 74LS245, U5 74LS253, U6 74LS253, U7 74LS253, U8 74LS253, U9 74LS253

Commit message: Finished a draft of the ALU PCB
Parts:
- removed J2: Interconnect 2, Connector_PinHeader_2.54mm:PinHeader_2x17_P2.54mm_Horizontal
- removed J3: Interconnect 3, Connector_PinHeader_2.54mm:PinHeader_2x17_P2.54mm_Horizontal
- added C44: 0.1uF, Capacitor_SMD:C_0603_1608Metric_Pad1.05x0.95mm_HandSolder, F.Cu at (64.8, 88.0)
- added C45: 0.1uF, Capacitor_SMD:C_0603_1608Metric_Pad1.05x0.95mm_HandSolder, F.Cu at (204.9, 77.1)
- added C46: 0.1uF, Capacitor_SMD:C_0603_1608Metric_Pad1.05x0.95mm_HandSolder, F.Cu at (181.1, 77.1)
- added C47: 0.1uF, Capacitor_SMD:C_0603_1608Metric_Pad1.05x0.95mm_HandSolder, F.Cu at (86.1, 46.7)
- added D33: overflow, LED_SMD:LED_1206_3216Metric_Pad1.42x1.75mm_HandSolder, F.Cu at (103.3, 30.7)
- added D34: sign, LED_SMD:LED_1206_3216Metric_Pad1.42x1.75mm_HandSolder, F.Cu at (106.3, 30.7)
- added D35: arithmetic_carry, LED_SMD:LED_1206_3216Metric_Pad1.42x1.75mm_HandSolder, F.Cu at (97.2, 30.7)
- added D36: logical_carry, LED_SMD:LED_1206_3216Metric_Pad1.42x1.75mm_HandSolder, F.Cu at (100.2, 30.7)
- added D37: zero, LED_SMD:LED_1206_3216Metric_Pad1.42x1.75mm_HandSolder, F.Cu at (109.3, 30.7)
- added R33: 220R, Resistor_SMD:R_0603_1608Metric_Pad1.05x0.95mm_HandSolder, F.Cu at (97.2, 36.6)
- added R34: 220R, Resistor_SMD:R_0603_1608Metric_Pad1.05x0.95mm_HandSolder, F.Cu at (100.2, 36.6)
- added R35: 220R, Resistor_SMD:R_0603_1608Metric_Pad1.05x0.95mm_HandSolder, F.Cu at (103.3, 36.6)
- added R36: 220R, Resistor_SMD:R_0603_1608Metric_Pad1.05x0.95mm_HandSolder, F.Cu at (106.3, 36.6)
- added R37: 220R, Resistor_SMD:R_0603_1608Metric_Pad1.05x0.95mm_HandSolder, F.Cu at (109.3, 36.6)
- added U47: 74LS245, Package_SO:SOIC-20W_7.5x12.8mm_P1.27mm, F.Cu at (86.2, 38.6)
- J1: value Interconnect 1 -> Interconnect; footprint Connector_PinHeader_2.54mm:PinHeader_2x17_P2.54mm_Horizontal -> Connector_PCBEdge:BUS_PCI
- TP1: value TestPoint -> GND
- TP10: value TestPoint -> HLT
- TP11: value TestPoint -> ~CLK
- TP12: value TestPoint -> CLK
- TP2: value TestPoint -> +5
- TP3: value TestPoint -> FLG Overflow
- TP4: value TestPoint -> FLG Sign
- TP5: value TestPoint -> FLG ArithCarry
- TP6: value TestPoint -> FLG LogCarry
- TP7: value TestPoint -> FLG Zero
- TP8: value TestPoint -> RST
- TP9: value TestPoint -> DBG
- moved C33 298.6 mm to (54.1, 71.5), turned to 180 degrees
- moved C21 298.5 mm to (54.1, 56.1), turned to 180 degrees
- moved C34 296.8 mm to (54.1, 86.9), turned to 180 degrees
- moved C22 296.2 mm to (64.8, 56.1), turned to 180 degrees
- moved U43 295.8 mm to (59.2, 99.1)
- moved U34 295.5 mm to (54.1, 80.8)
- moved U44 295.5 mm to (64.8, 81.3)
- moved U23 295.2 mm to (64.8, 65.4)
- moved U33 295.2 mm to (54.1, 65.4)
- moved U21 294.9 mm to (54.1, 50.0)
- moved U22 294.9 mm to (64.8, 50.0)
- moved C23 294.9 mm to (64.8, 71.5), turned to 180 degrees
- moved C11 282.7 mm to (54.1, 127.3), turned to 180 degrees
- moved C35 274.7 mm to (81.2, 74.4), turned to 180 degrees
- moved C42 271.7 mm to (75.9, 98.7), turned to 90 degrees
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Connections:
- C1 pad 2: Net-(C1-Pad2) -> GND
- C10 pad 2: Net-(C1-Pad2) -> GND
- C11 pad 2: Net-(C1-Pad2) -> GND
- C12 pad 2: Net-(C1-Pad2) -> GND
- C13 pad 2: Net-(C1-Pad2) -> GND
- C14 pad 2: Net-(C1-Pad2) -> GND
- C15 pad 2: Net-(C1-Pad2) -> GND
- C16 pad 2: Net-(C1-Pad2) -> GND
- C17 pad 2: Net-(C1-Pad2) -> GND
- C18 pad 2: Net-(C1-Pad2) -> GND
- C19 pad 2: Net-(C1-Pad2) -> GND
- C2 pad 2: Net-(C1-Pad2) -> GND
- C20 pad 2: Net-(C1-Pad2) -> GND
- C21 pad 2: Net-(C1-Pad2) -> GND
- C22 pad 2: Net-(C1-Pad2) -> GND
- C23 pad 2: Net-(C1-Pad2) -> GND
- C24 pad 2: Net-(C1-Pad2) -> GND
- C25 pad 2: Net-(C1-Pad2) -> GND
- C26 pad 2: Net-(C1-Pad2) -> GND
- C27 pad 2: Net-(C1-Pad2) -> GND
- C28 pad 2: Net-(C1-Pad2) -> GND
- C29 pad 2: Net-(C1-Pad2) -> GND
- C3 pad 2: Net-(C1-Pad2) -> GND
- C30 pad 2: Net-(C1-Pad2) -> GND
- C31 pad 2: Net-(C1-Pad2) -> GND
- C32 pad 2: Net-(C1-Pad2) -> GND
- C33 pad 2: Net-(C1-Pad2) -> GND
- C34 pad 2: Net-(C1-Pad2) -> GND
- C35 pad 2: Net-(C1-Pad2) -> GND
- C36 pad 2: Net-(C1-Pad2) -> GND
- C37 pad 2: Net-(C1-Pad2) -> GND
- C38 pad 2: Net-(C1-Pad2) -> GND
- C39 pad 2: Net-(C1-Pad2) -> GND
- C4 pad 2: Net-(C1-Pad2) -> GND
- C40 pad 2: Net-(C1-Pad2) -> GND
- C41 pad 2: Net-(C1-Pad2) -> GND
- C42 pad 2: Net-(C1-Pad2) -> GND
- C43 pad 2: Net-(C1-Pad2) -> GND
- C5 pad 2: Net-(C1-Pad2) -> GND
- C6 pad 2: Net-(C1-Pad2) -> GND
- C7 pad 2: Net-(C1-Pad2) -> GND
- C8 pad 2: Net-(C1-Pad2) -> GND
- C9 pad 2: Net-(C1-Pad2) -> GND
- D1 pad 1: Net-(D1-Pad1) -> GND
- D10 pad 1: Net-(D10-Pad1) -> GND
- D11 pad 1: Net-(D11-Pad1) -> GND
- D12 pad 1: Net-(D12-Pad1) -> GND
- D13 pad 1: Net-(D13-Pad1) -> GND
- D14 pad 1: Net-(D14-Pad1) -> GND
- D15 pad 1: Net-(D15-Pad1) -> GND
- D16 pad 1: Net-(D16-Pad1) -> GND
- D17 pad 1: Net-(D17-Pad1) -> GND
- D18 pad 1: Net-(D18-Pad1) -> GND
- D19 pad 1: Net-(D19-Pad1) -> GND
- D2 pad 1: Net-(D2-Pad1) -> GND
- D20 pad 1: Net-(D20-Pad1) -> GND
- D21 pad 1: Net-(D21-Pad1) -> GND
- D22 pad 1: Net-(D22-Pad1) -> GND
- D23 pad 1: Net-(D23-Pad1) -> GND
- D24 pad 1: Net-(D24-Pad1) -> GND
- D25 pad 1: Net-(D25-Pad1) -> GND
- D26 pad 1: Net-(D26-Pad1) -> GND
- D27 pad 1: Net-(D27-Pad1) -> GND
- D28 pad 1: Net-(D28-Pad1) -> GND
- D29 pad 1: Net-(D29-Pad1) -> GND
- D3 pad 1: Net-(D3-Pad1) -> GND
- D30 pad 1: Net-(D30-Pad1) -> GND
- D31 pad 1: Net-(D31-Pad1) -> GND
- D32 pad 1: Net-(D32-Pad1) -> GND
- D4 pad 1: Net-(D4-Pad1) -> GND
- D5 pad 1: Net-(D5-Pad1) -> GND
- D6 pad 1: Net-(D6-Pad1) -> GND
- D7 pad 1: Net-(D7-Pad1) -> GND
- D8 pad 1: Net-(D8-Pad1) -> GND
- D9 pad 1: Net-(D9-Pad1) -> GND
- R1 pad 1: Net-(D1-Pad1) -> Net-(R1-Pad1)
- R1 pad 2: +5V -> Net-(D1-Pad2)
- R10 pad 1: Net-(D10-Pad1) -> Net-(R10-Pad1)
- R10 pad 2: +5V -> Net-(D10-Pad2)
- R11 pad 1: Net-(D11-Pad1) -> Net-(R11-Pad1)
- R11 pad 2: +5V -> Net-(D11-Pad2)
- R12 pad 1: Net-(D12-Pad1) -> Net-(R12-Pad1)
- R12 pad 2: +5V -> Net-(D12-Pad2)
- R13 pad 1: Net-(D13-Pad1) -> Net-(R13-Pad1)
- R13 pad 2: +5V -> Net-(D13-Pad2)
- R14 pad 1: Net-(D14-Pad1) -> Net-(R14-Pad1)
- R14 pad 2: +5V -> Net-(D14-Pad2)
- R15 pad 1: Net-(D15-Pad1) -> Net-(R15-Pad1)
- R15 pad 2: +5V -> Net-(D15-Pad2)
- R16 pad 1: Net-(D16-Pad1) -> Net-(R16-Pad1)
- R16 pad 2: +5V -> Net-(D16-Pad2)
- R17 pad 1: Net-(D17-Pad1) -> Net-(R17-Pad1)
- R17 pad 2: +5V -> Net-(D17-Pad2)
- R18 pad 1: Net-(D18-Pad1) -> Net-(R18-Pad1)
- R18 pad 2: +5V -> Net-(D18-Pad2)
- R19 pad 1: Net-(D19-Pad1) -> Net-(R19-Pad1)
- R19 pad 2: +5V -> Net-(D19-Pad2)
- R2 pad 1: Net-(D2-Pad1) -> Net-(R2-Pad1)
- R2 pad 2: +5V -> Net-(D2-Pad2)
- R20 pad 1: Net-(D20-Pad1) -> Net-(R20-Pad1)
- R20 pad 2: +5V -> Net-(D20-Pad2)
- R21 pad 1: Net-(D21-Pad1) -> Net-(R21-Pad1)
- R21 pad 2: +5V -> Net-(D21-Pad2)
- R22 pad 1: Net-(D22-Pad1) -> Net-(R22-Pad1)
- R22 pad 2: +5V -> Net-(D22-Pad2)
- R23 pad 1: Net-(D23-Pad1) -> Net-(R23-Pad1)
- R23 pad 2: +5V -> Net-(D23-Pad2)
- R24 pad 1: Net-(D24-Pad1) -> Net-(R24-Pad1)
- R24 pad 2: +5V -> Net-(D24-Pad2)
- R25 pad 1: Net-(D25-Pad1) -> Net-(R25-Pad1)
- R25 pad 2: +5V -> Net-(D25-Pad2)
- R26 pad 1: Net-(D26-Pad1) -> Net-(R26-Pad1)
- R26 pad 2: +5V -> Net-(D26-Pad2)
- R27 pad 1: Net-(D27-Pad1) -> Net-(R27-Pad1)
- R27 pad 2: +5V -> Net-(D27-Pad2)
- R28 pad 1: Net-(D28-Pad1) -> Net-(R28-Pad1)
- R28 pad 2: +5V -> Net-(D28-Pad2)
- R29 pad 1: Net-(D29-Pad1) -> Net-(R29-Pad1)
- R29 pad 2: +5V -> Net-(D29-Pad2)
- R3 pad 1: Net-(D3-Pad1) -> Net-(R3-Pad1)
- R3 pad 2: +5V -> Net-(D3-Pad2)
- R30 pad 1: Net-(D30-Pad1) -> Net-(R30-Pad1)
- R30 pad 2: +5V -> Net-(D30-Pad2)
- R31 pad 1: Net-(D31-Pad1) -> Net-(R31-Pad1)
- R31 pad 2: +5V -> Net-(D31-Pad2)
- R32 pad 1: Net-(D32-Pad1) -> Net-(R32-Pad1)
- R32 pad 2: +5V -> Net-(D32-Pad2)
- R4 pad 1: Net-(D4-Pad1) -> Net-(R4-Pad1)
- R4 pad 2: +5V -> Net-(D4-Pad2)
- R5 pad 1: Net-(D5-Pad1) -> Net-(R5-Pad1)
- R5 pad 2: +5V -> Net-(D5-Pad2)
- R6 pad 1: Net-(D6-Pad1) -> Net-(R6-Pad1)
- R6 pad 2: +5V -> Net-(D6-Pad2)
- R7 pad 1: Net-(D7-Pad1) -> Net-(R7-Pad1)
- R7 pad 2: +5V -> Net-(D7-Pad2)
- R8 pad 1: Net-(D8-Pad1) -> Net-(R8-Pad1)
- R8 pad 2: +5V -> Net-(D8-Pad2)
- R9 pad 1: Net-(D9-Pad1) -> Net-(R9-Pad1)
- R9 pad 2: +5V -> Net-(D9-Pad2)
- TP1 pad 1: +5V -> GND
- U1 pad 10: +5V -> GND
- U1 pad 11: Net-(D15-Pad2) -> Net-(R15-Pad1)
- U1 pad 12: Net-(D13-Pad2) -> Net-(R13-Pad1)
- U1 pad 13: Net-(D11-Pad2) -> Net-(R11-Pad1)
- U1 pad 14: Net-(D9-Pad2) -> Net-(R9-Pad1)
- U1 pad 15: Net-(D7-Pad2) -> Net-(R7-Pad1)
- U1 pad 16: Net-(D5-Pad2) -> Net-(R5-Pad1)
- U1 pad 17: Net-(D3-Pad2) -> Net-(R3-Pad1)
- U1 pad 18: Net-(D1-Pad2) -> Net-(R1-Pad1)
- U10 pad 1: +5V -> GND
- U10 pad 8: +5V -> GND
- U11 pad 1: +5V -> GND
- U11 pad 8: +5V -> GND
- U12 pad 1: +5V -> GND
- U12 pad 8: +5V -> GND
- U13 pad 1: +5V -> GND
- U13 pad 8: +5V -> GND
- U14 pad 1: +5V -> GND
- U14 pad 8: +5V -> GND
- U15 pad 1: +5V -> GND
- U15 pad 8: +5V -> GND
- U16 pad 1: +5V -> GND
- U16 pad 8: +5V -> GND
- U17 pad 1: +5V -> GND
- U17 pad 8: +5V -> GND
- U18 pad 1: +5V -> GND
- U18 pad 8: +5V -> GND
- U19 pad 10: +5V -> GND
- U19 pad 11: Net-(D31-Pad2) -> Net-(R31-Pad1)
- U19 pad 12: Net-(D29-Pad2) -> Net-(R29-Pad1)
- U19 pad 13: Net-(D27-Pad2) -> Net-(R27-Pad1)
- U19 pad 14: Net-(D25-Pad2) -> Net-(R25-Pad1)
- U19 pad 15: Net-(D23-Pad2) -> Net-(R23-Pad1)
- U19 pad 16: Net-(D21-Pad2) -> Net-(R21-Pad1)
- U19 pad 17: Net-(D19-Pad2) -> Net-(R19-Pad1)
- U19 pad 18: Net-(D17-Pad2) -> Net-(R17-Pad1)
- U2 pad 10: +5V -> GND
- U2 pad 11: Net-(D16-Pad2) -> Net-(R16-Pad1)
- U2 pad 12: Net-(D14-Pad2) -> Net-(R14-Pad1)
- U2 pad 13: Net-(D12-Pad2) -> Net-(R12-Pad1)
- U2 pad 14: Net-(D10-Pad2) -> Net-(R10-Pad1)
- U2 pad 15: Net-(D8-Pad2) -> Net-(R8-Pad1)
- U2 pad 16: Net-(D6-Pad2) -> Net-(R6-Pad1)
- U2 pad 17: Net-(D4-Pad2) -> Net-(R4-Pad1)
- U2 pad 18: Net-(D2-Pad2) -> Net-(R2-Pad1)
- U20 pad 10: +5V -> GND
- U20 pad 11: Net-(D32-Pad2) -> Net-(R32-Pad1)
- U20 pad 12: Net-(D30-Pad2) -> Net-(R30-Pad1)
- U20 pad 13: Net-(D28-Pad2) -> Net-(R28-Pad1)
- U20 pad 14: Net-(D26-Pad2) -> Net-(R26-Pad1)
- U20 pad 15: Net-(D24-Pad2) -> Net-(R24-Pad1)
- U20 pad 16: Net-(D22-Pad2) -> Net-(R22-Pad1)
- U20 pad 17: Net-(D20-Pad2) -> Net-(R20-Pad1)
- U20 pad 18: Net-(D18-Pad2) -> Net-(R18-Pad1)
- U21 pad 7: +5V -> GND
- U22 pad 7: +5V -> GND
- U23 pad 7: +5V -> GND
- U24 pad 1: +5V -> GND
- U24 pad 13: +5V -> GND
- U24 pad 15: +5V -> GND
- U24 pad 3: +5V -> GND
- U24 pad 8: +5V -> GND
- U25 pad 1: +5V -> GND
- U25 pad 13: +5V -> GND
- U25 pad 15: +5V -> GND
- U25 pad 3: +5V -> GND
- U25 pad 8: +5V -> GND
- U26 pad 1: +5V -> GND
- U26 pad 13: +5V -> GND
- U26 pad 15: +5V -> GND
- U26 pad 3: +5V -> GND
- U26 pad 8: +5V -> GND
- U27 pad 1: +5V -> GND
- U27 pad 13: +5V -> GND
- U27 pad 15: +5V -> GND
- U27 pad 3: +5V -> GND
- U27 pad 8: +5V -> GND
- U28 pad 1: +5V -> GND
- U28 pad 13: +5V -> GND
- U28 pad 15: +5V -> GND
- U28 pad 3: +5V -> GND
- U28 pad 8: +5V -> GND
- U29 pad 1: +5V -> GND
- U29 pad 13: +5V -> GND
- U29 pad 15: +5V -> GND
- U29 pad 3: +5V -> GND
- U29 pad 8: +5V -> GND
- U3 pad 1: +5V -> GND
- U3 pad 8: +5V -> GND
- U30 pad 1: +5V -> GND
- U30 pad 13: +5V -> GND
- U30 pad 15: +5V -> GND
- U30 pad 3: +5V -> GND
- U30 pad 8: +5V -> GND
- U31 pad 1: +5V -> GND
- U31 pad 13: +5V -> GND
- U31 pad 15: +5V -> GND
- U31 pad 3: +5V -> GND
- U31 pad 8: +5V -> GND
- U32 pad 1: +5V -> GND
- U32 pad 10: +5V -> GND
- U32 pad 13: +5V -> GND
- U32 pad 15: +5V -> GND
- U32 pad 3: +5V -> GND
- U32 pad 4: +5V -> GND
- U32 pad 5: +5V -> GND
- U32 pad 6: +5V -> GND
- U32 pad 8: +5V -> GND
- U33 pad 7: +5V -> GND
- U34 pad 7: +5V -> GND
- U35 pad 8: +5V -> GND
- U36 pad 8: +5V -> GND
- U37 pad 8: +5V -> GND
- U38 pad 8: +5V -> GND
- U39 pad 1: +5V -> GND
- U39 pad 10: +5V -> GND
- U4 pad 1: +5V -> GND
- U4 pad 8: +5V -> GND
- U40 pad 1: +5V -> GND
- U40 pad 10: +5V -> GND
- U41 pad 1: +5V -> GND
- U41 pad 10: +5V -> GND
- U42 pad 1: +5V -> GND
- U42 pad 10: +5V -> GND
- U43 pad 1: +5V -> GND
- U43 pad 10: +5V -> GND
- U43 pad 18: /arrithmetic_carry_flag -> /arithmetic_carry_flag
- U44 pad 10: +5V -> GND
- U44 pad 11: /arrithmetic_carry_flag -> /arithmetic_carry_flag
- U44 pad 13: +5V -> GND
- U44 pad 15: +5V -> GND
- U44 pad 8: +5V -> GND
- U45 pad 10: +5V -> GND
- U46 pad 10: +5V -> GND
- U5 pad 1: +5V -> GND
- U5 pad 8: +5V -> GND
- U6 pad 1: +5V -> GND
- U6 pad 8: +5V -> GND
- U7 pad 1: +5V -> GND
- U7 pad 8: +5V -> GND
- U8 pad 1: +5V -> GND
- U8 pad 8: +5V -> GND
- U9 pad 1: +5V -> GND
- U9 pad 8: +5V -> GND
Routing:
- net GND: track 0.00 -> 2113.9 mm, vias 0 -> 76
- net +5V: track 0.00 -> 1589.6 mm, vias 0 -> 63
- net /bit_control_1: track 0.00 -> 521.4 mm, vias 0 -> 17
- net /y_bus_14: track 0.00 -> 445.7 mm, vias 0 -> 16
- net /add_15: track 0.00 -> 390.7 mm, vias 0 -> 9
- net /CLK: track 0.00 -> 363.8 mm, vias 0 -> 12
- net /y_bus_02: track 0.00 -> 345.3 mm, vias 0 -> 13
- net /bit_control_3: track 0.00 -> 335.7 mm, vias 0 -> 21
- net /d_bus_13: track 0.00 -> 331.1 mm, vias 0 -> 6
- net /logical_carry_flag: track 0.00 -> 330.5 mm, vias 0 -> 8
- net /shift_control_0: track 0.00 -> 326.1 mm, vias 0 -> 27
- net /y_bus_01: track 0.00 -> 319.8 mm, vias 0 -> 12
- net /y_bus_00: track 0.00 -> 307.9 mm, vias 0 -> 9
- net /x_bus_00: track 0.00 -> 296.3 mm, vias 0 -> 7
- net /y_bus_03: track 0.00 -> 293.6 mm, vias 0 -> 7
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Other:
- board outline added: 177 x 121.9 mm
- board text added: "15 14 13 12 11 10 9 8"
- board text added: "7 6 5 4 3 2 1 0"
- board text added: "Flags"
- board text added: "Y Bus"

Commit message: Upgrade to KiCad 6 and commit a bunch of random stuff
Parts:
- TP11: value ~CLK -> ~{CLK}
Connections:
- net /~CLK renamed /~{CLK}
Other:
- net class Default removed
