File: cpu/Backplane/Backplane.sch (KiCad schematic (older format))
At the start: 1 part

Commit message: Lots of changes
Parts:
- removed J?: Conn_02x34_Odd_Even, symbol Connector_Generic:Conn_02x34_Odd_Even
- added C1, C2, C3, C4, C5, C6, C7, C8: 0.1uF, Capacitor_SMD:C_0603_1608Metric_Pad1.05x0.95mm_HandSolder, symbol Device:C
- added D0, D1, D10, D11, D12, D13, D14, D15, D16, D17, D18, D19, D2, D20, D21, D22, D23, D24, D25, D26, D27, D28, D29, D3, D30, D31, D32, D33, D34, D35, D36, D37, D38, D39, D4, D40, D41, D42, D43, D44, D45, D46, D47, D48, D49, D5, D50, D51, D52, D53, D54, D55, D56, D57, D58, D59, D6, D60, D61, D62, D63, D7, D8, D9: LED_BLUE, LED_SMD:LED_1206_3216Metric_Pad1.42x1.75mm_HandSolder, symbol Device:LED_ALT
- added J1: GPR A1, Connector_PinHeader_2.54mm:PinHeader_2x17_P2.54mm_Vertical, symbol Connector_Generic:Conn_02x17_Odd_Even
- added J10: SI 2, Connector_PinHeader_2.54mm:PinHeader_2x17_P2.54mm_Vertical, symbol Connector_Generic:Conn_02x17_Odd_Even
- added J11: DI 1, Connector_PinHeader_2.54mm:PinHeader_2x17_P2.54mm_Vertical, symbol Connector_Generic:Conn_02x17_Odd_Even
- added J12: DI 2, Connector_PinHeader_2.54mm:PinHeader_2x17_P2.54mm_Vertical, symbol Connector_Generic:Conn_02x17_Odd_Even
- added J13: SP 1, Connector_PinHeader_2.54mm:PinHeader_2x17_P2.54mm_Vertical, symbol Connector_Generic:Conn_02x17_Odd_Even
- added J14: SP 2, Connector_PinHeader_2.54mm:PinHeader_2x17_P2.54mm_Vertical, symbol Connector_Generic:Conn_02x17_Odd_Even
- added J15: PC 1, Connector_PinHeader_2.54mm:PinHeader_2x17_P2.54mm_Vertical, symbol Connector_Generic:Conn_02x17_Odd_Even
- added J16: PC 2, Connector_PinHeader_2.54mm:PinHeader_2x17_P2.54mm_Vertical, symbol Connector_Generic:Conn_02x17_Odd_Even
- added J17: HOLDING 1, Connector_PinHeader_2.54mm:PinHeader_2x17_P2.54mm_Vertical, symbol Connector_Generic:Conn_02x17_Odd_Even
- added J18: HOLDING 2, Connector_PinHeader_2.54mm:PinHeader_2x17_P2.54mm_Vertical, symbol Connector_Generic:Conn_02x17_Odd_Even
- added J2: GPR A2, Connector_PinHeader_2.54mm:PinHeader_2x17_P2.54mm_Vertical, symbol Connector_Generic:Conn_02x17_Odd_Even
- added J3: GPR B1, Connector_PinHeader_2.54mm:PinHeader_2x17_P2.54mm_Vertical, symbol Connector_Generic:Conn_02x17_Odd_Even
- added J4: GPR B2, Connector_PinHeader_2.54mm:PinHeader_2x17_P2.54mm_Vertical, symbol Connector_Generic:Conn_02x17_Odd_Even
- added J5: GPR C1, Connector_PinHeader_2.54mm:PinHeader_2x17_P2.54mm_Vertical, symbol Connector_Generic:Conn_02x17_Odd_Even
- added J6: GPR C2, Connector_PinHeader_2.54mm:PinHeader_2x17_P2.54mm_Vertical, symbol Connector_Generic:Conn_02x17_Odd_Even
- added J7: GPR D1, Connector_PinHeader_2.54mm:PinHeader_2x17_P2.54mm_Vertical, symbol Connector_Generic:Conn_02x17_Odd_Even
- added J8: GPR D2, Connector_PinHeader_2.54mm:PinHeader_2x17_P2.54mm_Vertical, symbol Connector_Generic:Conn_02x17_Odd_Even
- added J9: SI 1, Connector_PinHeader_2.54mm:PinHeader_2x17_P2.54mm_Vertical, symbol Connector_Generic:Conn_02x17_Odd_Even
- added R0, R1, R10, R11, R12, R13, R14, R15, R16, R17, R18, R19, R2, R20, R21, R22, R23, R24, R25, R26, R27, R28, R29, R3, R30, R31, R32, R33, R34, R35, R36, R37, R38, R39, R4, R40, R41, R42, R43, R44, R45, R46, R47, R48, R49, R5, R50, R51, R52, R53, R54, R55, R56, R57, R58, R59, R6, R60, R61, R62, R63, R7, R8, R9: 220R, Resistor_SMD:R_0603_1608Metric_Pad1.05x0.95mm_HandSolder, symbol Device:R
- added U1, U2, U3, U4, U5, U6, U7, U8: 74LS245, Package_SO:SOIC-20W_7.5x12.8mm_P1.27mm, symbol 74xx:74LS245
Connections:
- net labels added: +5V, CLK, GND, HLT, RST, a_bus_00, a_bus_01, a_bus_02, a_bus_03, a_bus_04, a_bus_05, a_bus_06, a_bus_07, a_bus_08, a_bus_09, a_bus_10, a_bus_11, a_bus_12, a_bus_13, a_bus_14, a_bus_15, a_bus_write_di, a_bus_write_pc, a_bus_write_si, d_bus_00, d_bus_01, d_bus_02, d_bus_03, d_bus_04, d_bus_05, d_bus_06, d_bus_07, d_bus_08, d_bus_09, d_bus_10, d_bus_11, d_bus_12, d_bus_13, d_bus_14, d_bus_15, d_bus_read_di, d_bus_read_gpr_a, d_bus_read_gpr_b, d_bus_read_gpr_c, d_bus_read_gpr_d, d_bus_read_pc, d_bus_read_si, d_bus_write_di, d_bus_write_gpr_a, d_bus_write_gpr_b, d_bus_write_gpr_c, d_bus_write_gpr_d, d_bus_write_pc, d_bus_write_si, reg_borrow_di, reg_borrow_pc, reg_borrow_si, reg_borrow_sp, reg_carry_di, reg_carry_pc, reg_carry_si, reg_carry_sp, reg_dec_di, reg_dec_pc, reg_dec_si, reg_inc_di, reg_inc_pc, reg_inc_si, x_bus_00, x_bus_01, x_bus_02, x_bus_03, x_bus_04, x_bus_05, x_bus_06, x_bus_07, x_bus_08, x_bus_09, x_bus_10, x_bus_11, x_bus_12, x_bus_13, x_bus_14, x_bus_15, x_bus_write_gpr_a, x_bus_write_gpr_b, x_bus_write_gpr_c, x_bus_write_gpr_d, y_bus_00, y_bus_01, y_bus_02, y_bus_03, y_bus_04, y_bus_05, y_bus_06, y_bus_07, y_bus_08, y_bus_09, y_bus_10, y_bus_11, y_bus_12, y_bus_13, y_bus_14, y_bus_15, y_bus_write_gpr_a, y_bus_write_gpr_b, y_bus_write_gpr_c, y_bus_write_gpr_d, ~CLK, ~DBG
- wire segments 0 -> 1160
- no-connect marks 0 -> 144
Other:
- note added: "Address Registers"
- note added: "General Purpose Registers"

Commit message: Added missing power pins to GPR
Parts:
- removed J1: GPR A1, Connector_PinHeader_2.54mm:PinHeader_2x17_P2.54mm_Vertical, symbol Connector_Generic:Conn_02x17_Odd_Even
- removed J2: GPR A2, Connector_PinHeader_2.54mm:PinHeader_2x17_P2.54mm_Vertical, symbol Connector_Generic:Conn_02x17_Odd_Even
- added J1: GPR_A, TE-PCI-32bit:TE_1-5145154-2, symbol cpu_custom_symbols:Bus_PCI_32bit_5V
- added U?: 74LS245_BiDirection, symbol cpu_custom_symbols:74LS245_BiDirection
Connections:
- wire segments 1160 -> 1112
- no-connect marks 144 -> 187

Commit message: Upgrade to KiCad 6 and commit a bunch of random stuff
Parts:
- removed J10: SI 2, Connector_PinHeader_2.54mm:PinHeader_2x17_P2.54mm_Vertical, symbol Connector_Generic:Conn_02x17_Odd_Even
- removed J11: DI 1, Connector_PinHeader_2.54mm:PinHeader_2x17_P2.54mm_Vertical, symbol Connector_Generic:Conn_02x17_Odd_Even
- removed J12: DI 2, Connector_PinHeader_2.54mm:PinHeader_2x17_P2.54mm_Vertical, symbol Connector_Generic:Conn_02x17_Odd_Even
- removed J13: SP 1, Connector_PinHeader_2.54mm:PinHeader_2x17_P2.54mm_Vertical, symbol Connector_Generic:Conn_02x17_Odd_Even
- removed J14: SP 2, Connector_PinHeader_2.54mm:PinHeader_2x17_P2.54mm_Vertical, symbol Connector_Generic:Conn_02x17_Odd_Even
- removed J15: PC 1, Connector_PinHeader_2.54mm:PinHeader_2x17_P2.54mm_Vertical, symbol Connector_Generic:Conn_02x17_Odd_Even
- removed J16: PC 2, Connector_PinHeader_2.54mm:PinHeader_2x17_P2.54mm_Vertical, symbol Connector_Generic:Conn_02x17_Odd_Even
- removed J17: HOLDING 1, Connector_PinHeader_2.54mm:PinHeader_2x17_P2.54mm_Vertical, symbol Connector_Generic:Conn_02x17_Odd_Even
- removed J18: HOLDING 2, Connector_PinHeader_2.54mm:PinHeader_2x17_P2.54mm_Vertical, symbol Connector_Generic:Conn_02x17_Odd_Even
- removed J3: GPR B1, Connector_PinHeader_2.54mm:PinHeader_2x17_P2.54mm_Vertical, symbol Connector_Generic:Conn_02x17_Odd_Even
- removed J4: GPR B2, Connector_PinHeader_2.54mm:PinHeader_2x17_P2.54mm_Vertical, symbol Connector_Generic:Conn_02x17_Odd_Even
- removed J5: GPR C1, Connector_PinHeader_2.54mm:PinHeader_2x17_P2.54mm_Vertical, symbol Connector_Generic:Conn_02x17_Odd_Even
- removed J6: GPR C2, Connector_PinHeader_2.54mm:PinHeader_2x17_P2.54mm_Vertical, symbol Connector_Generic:Conn_02x17_Odd_Even
- removed J7: GPR D1, Connector_PinHeader_2.54mm:PinHeader_2x17_P2.54mm_Vertical, symbol Connector_Generic:Conn_02x17_Odd_Even
- removed J8: GPR D2, Connector_PinHeader_2.54mm:PinHeader_2x17_P2.54mm_Vertical, symbol Connector_Generic:Conn_02x17_Odd_Even
- removed J9: SI 1, Connector_PinHeader_2.54mm:PinHeader_2x17_P2.54mm_Vertical, symbol Connector_Generic:Conn_02x17_Odd_Even
- removed R0, R1, R10, R11, R12, R13, R14, R15, R16, R17, R18, R19, R2, R20, R21, R22, R23, R24, R25, R26, R27, R28, R29, R3, R30, R31, R32, R33, R34, R35, R36, R37, R38, R39, R4, R40, R41, R42, R43, R44, R45, R46, R47, R48, R49, R5, R50, R51, R52, R53, R54, R55, R56, R57, R58, R59, R6, R60, R61, R62, R63, R7, R8, R9: 220R, Resistor_SMD:R_0603_1608Metric_Pad1.05x0.95mm_HandSolder, symbol Device:R
- removed U1, U2, U3, U4, U5, U6, U7, U8: 74LS245, Package_SO:SOIC-20W_7.5x12.8mm_P1.27mm, symbol 74xx:74LS245
- added C10, C11, C12, C13, C14, C15, C16, C17, C18, C19, C20, C21, C22, C23, C24, C25: 47uF, Capacitor_SMD:CP_Elec_4x5.4, symbol Device:CP1
- added C9: 0.1uF, Capacitor_SMD:C_0603_1608Metric_Pad1.05x0.95mm_HandSolder, symbol Device:C
- added D64: D_Zener, Diode_THT:D_A-405_P10.16mm_Horizontal, symbol Device:D_Zener
- added J10: ALU, TE-PCI-32bit:TE_1-5145154-2, symbol cpu_custom_symbols:Bus_PCI_32bit_5V
- added J11: Memory, TE-PCI-32bit:TE_1-5145154-2, symbol cpu_custom_symbols:Bus_PCI_32bit_5V
- added J12, J13, J14, J15: Conn_01x16_Female, Connector_PinHeader_2.54mm:PinHeader_1x16_P2.54mm_Vertical, symbol Connector:Conn_01x16_Female
- added J16, J17, J18, J19, J27: Conn_01x04_Female, Connector_PinHeader_2.54mm:PinHeader_1x04_P2.54mm_Vertical, symbol Connector:Conn_01x04_Female
- added J2: GPR_B, TE-PCI-32bit:TE_1-5145154-2, symbol cpu_custom_symbols:Bus_PCI_32bit_5V
- added J20, J21, J22, J23: Conn_01x07_Female, Connector_PinHeader_2.54mm:PinHeader_1x07_P2.54mm_Vertical, symbol Connector:Conn_01x07_Female
- added J24: Conn_01x05_Female, Connector_PinHeader_2.54mm:PinHeader_1x05_P2.54mm_Vertical, symbol Connector:Conn_01x05_Female
- added J25: Barrel_Jack, digikey-footprints:Barrel_Jack_5.5mmODx2.1mmID_PJ-202A, symbol Connector:Barrel_Jack
- added J28: Conn_01x14_Female, Connector_PinHeader_2.54mm:PinHeader_1x14_P2.54mm_Vertical, symbol Connector:Conn_01x14_Female
- added J29: IO_1, TE-PCI-32bit:TE_1-5145154-2, symbol cpu_custom_symbols:Bus_PCI_32bit_5V
- added J3: GPR_C, TE-PCI-32bit:TE_1-5145154-2, symbol cpu_custom_symbols:Bus_PCI_32bit_5V
- added J30: IO_2, TE-PCI-32bit:TE_1-5145154-2, symbol cpu_custom_symbols:Bus_PCI_32bit_5V
- added J31: IO_3, TE-PCI-32bit:TE_1-5145154-2, symbol cpu_custom_symbols:Bus_PCI_32bit_5V
- added J32: IO_4, TE-PCI-32bit:TE_1-5145154-2, symbol cpu_custom_symbols:Bus_PCI_32bit_5V
- added J4: GPR_D, TE-PCI-32bit:TE_1-5145154-2, symbol cpu_custom_symbols:Bus_PCI_32bit_5V
- added J5: AReg_PC, TE-PCI-32bit:TE_1-5145154-2, symbol cpu_custom_symbols:Bus_PCI_32bit_5V
- added J6: AReg_SP, TE-PCI-32bit:TE_1-5145154-2, symbol cpu_custom_symbols:Bus_PCI_32bit_5V
- added J7: AReg_SI, TE-PCI-32bit:TE_1-5145154-2, symbol cpu_custom_symbols:Bus_PCI_32bit_5V
- added J8: AReg_DI, TE-PCI-32bit:TE_1-5145154-2, symbol cpu_custom_symbols:Bus_PCI_32bit_5V
- added J9: Pipeline, TE-PCI-32bit:TE_1-5145154-2, symbol cpu_custom_symbols:Bus_PCI_32bit_5V
- added RN1, RN2, RN3, RN4, RN5, RN6, RN7, RN8: 220R, Resistor_SMD:R_Array_Convex_8x0602, symbol Device:R_Pack08
- added U1, U2, U3, U4, U6, U7, U8: 74LS245, Package_SO:SOIC-20W_7.5x12.8mm_P1.27mm, symbol cpu_custom_symbols:74LS245_BiDirection
- added U10: 74LS04, Package_SO:SOIC-14_3.9x8.7mm_P1.27mm, symbol 74xx:74LS04
- added U9: MCP100-450D, digikey-footprints:SOT-23-3, symbol Power_Supervisor:MCP100-450D
- U5: renamed from U?; value 74LS245_BiDirection -> 74LS245; footprint (none) -> Package_SO:SOIC-20W_7.5x12.8mm_P1.27mm
Connections:
- net labels added: BANK, MEM_RD, MEM_WR, MREQ, a_bus_write_sp, alu_arr_carry_sel_0, alu_arr_carry_sel_1, alu_bit_control_0, alu_bit_control_1, alu_bit_control_2, alu_bit_control_3, alu_shift_control_0, alu_shift_control_1, arrithmetic_carry_flag, d_bus_read_sp, d_bus_write_alu, d_bus_write_sp, logical_carry_flag, md_bus_00, md_bus_01, md_bus_02, md_bus_03, md_bus_04, md_bus_05, md_bus_06, md_bus_07, md_bus_08, md_bus_09, md_bus_10, md_bus_11, md_bus_12, md_bus_13, md_bus_14, md_bus_15, overflow_flag, reg_dec_sp, reg_inc_sp, sign_flag, zero_flag
- wire segments 1112 -> 1649
- no-connect marks 187 -> 851
Other:
- moved on the sheet: C1, D0, D1, D10, D11, D12, D13, D14, D15, D16, D17, D18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
