File: cpu/BreakOutBoard/BreakOutBoard.kicad_pcb (KiCad board)
At the start: 2 copper layers, 156.2 x 45.6 mm, 12 parts, among them J1 Conn_01x01_Male, J10 Conn_01x16_Male, J11 Conn_01x07_Male, J12 Conn_01x07_Male, J2 Conn_01x01_Male, J3 Conn_01x02_Male, J4 Conn_01x16_Male, J5 Conn_01x16_Male, J6 Conn_01x16_Male, J7 Conn_01x16_Male, J8 Bus_PCI_32bit_5V, J9 Conn_01x16_Male

Commit message: Upgrade to KiCad 6 and commit a bunch of random stuff
Connections:
- net /~CLK renamed /~{CLK}
Other:
- net class Default removed
- board text added: "~{CLK}"
- board text added: "~{DBG}"
- board text removed: "~CLK"
- board text removed: "~DBG"
