File: cpu/AddressRegister/AddressRegisterModule.kicad_sch (KiCad schematic)
At the start: 61 parts, among them J1 Bus_PCI_32bit_5V, U1 74LS193, U10 74LS245, U11 74LS245, U12 74LS00, U2 74LS193, U3 74LS193, U4 74LS193, U5 74LS245, U6 74LS245, U7 74LS245, U8 74LS245, U9 74LS245

Commit message: Address Register v1.3
Parts:
- C13, C14: symbol Device:CP1 -> Device:C_Polarized_US
- D1, D10, D17, D18, D19, D2, D20, D21, D22, D23, D3, D4, D5, D6, D7, D8, D9: symbol Device:D_ALT -> Device:LED_Filled
- D11, D12, D13, D14, D15, D16: symbol Device:LED_ALT -> Device:LED_Filled
- R1, R2, R3, R4, R5, R6, R7, R8: renamed from R?; footprint (none) -> Resistor_SMD:R_0603_1608Metric_Pad0.98x0.95mm_HandSolder
Connections:
- net HLT: no longer names the net of J1.B58 (HLT)
- net ~{CLK}: no longer names the net of J1.B59 (~{CLK})
