File: cpu/AddressRegister/AddressRegisterModule.sch (KiCad schematic (older format))
At the start: 71 parts, among them J1 Interconnect, U1 74LS193, U10 74LS245, U11 74LS245, U12 74LS00, U2 74LS193, U3 74LS193, U4 74LS193, U5 74LS245, U6 74LS245, U7 74LS245, U8 74LS245, U9 74LS245

Commit message: Finished Address Register 1.0
Parts:
- removed J1: Interconnect, Connector_PCBEdge:BUS_PCI, symbol MySymbols:Bus_PCI_32bit_5V
- removed R1, R10, R11, R12, R13, R14, R15, R16, R17, R18, R19, R2, R20, R21, R22, R23, R3, R4, R5, R6, R7, R8, R9: 220R, Resistor_SMD:R_0603_1608Metric_Pad1.05x0.95mm_HandSolder, symbol Device:R
- removed U10, U11, U5, U6, U7, U8, U9: 74LS245, Package_SO:SOIC-20W_7.5x12.8mm_P1.27mm, symbol CounterRegisterModule-rescue:74LS245_BiDirection-74ls245_bidirection
- added C13, C14: 10uF, Capacitor_SMD:CP_Elec_4x5.4, symbol Device:CP1
- added J1: Bus_PCI_32bit_5V, Connector_PCBEdge:BUS_PCI, symbol cpu_custom_symbols:Bus_PCI_32bit_5V
- added RN1, RN2, RN3: 220R, Resistor_SMD:R_Array_Convex_8x0602, symbol Device:R_Pack08
- added U10, U11, U5, U6, U7, U8, U9: 74LS245, Package_SO:SOIC-20W_7.5x12.8mm_P1.27mm, symbol cpu_custom_symbols:74LS245_BiDirection
- D1, D10, D11, D12, D13, D14, D15, D16, D2, D3, D4, D5, D6, D7, D8, D9: Digikey 732-4978-1-ND -> 732-4991-1-ND
- D17, D18, D19, D20, D21, D22, D23: Digikey 732-4988-1-ND -> 732-4994-1-ND
Connections:
- wire segments 540 -> 551
- no-connect marks 75 -> 77
Other:
- moved on the sheet: D1, D10, D11, D12, D13, D14, D15, D16, D17, D18, D19, D2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

Commit message: Address Register v1.3
Parts:
- C13, C14: symbol Device:CP1 -> Device:C_Polarized_US
- D1, D10, D17, D18, D19, D2, D20, D21, D22, D23, D3, D4, D5, D6, D7, D8, D9: symbol Device:D_ALT -> Device:LED_Filled
- D11, D12, D13, D14, D15, D16: symbol Device:LED_ALT -> Device:LED_Filled
Changed lines of the file:
@@
 	12800 1550 12800 1750
 $Comp
-L Device:D_ALT D1
+L Device:LED_Filled D1
 U 1 1 5F39D1DC
 P 12600 3150
@@
 $EndComp
 $Comp
-L Device:D_ALT D2
+L Device:LED_Filled D2
 U 1 1 5F3A1909
 P 12800 3150
@@
 $EndComp
 $Comp
-L Device:D_ALT D3
+L Device:LED_Filled D3
 U 1 1 5F3BD052
 P 13000 3150
@@
 $EndComp
 $Comp
-L Device:D_ALT D4
+L Device:LED_Filled D4
 U 1 1 5F3BD066
 P 13200 3150
@@
 $EndComp
 $Comp
-L Device:D_ALT D5
+L Device:LED_Filled D5
 U 1 1 5F41313D
 P 13400 3150
@@
 $EndComp
 $Comp
-L Device:D_ALT D6
+L Device:LED_Filled D6
 U 1 1 5F413151
 P 13600 3150
@@
 $EndComp
 $Comp
-L Device:D_ALT D7
+L Device:LED_Filled D7
 U 1 1 5F413165
 P 13800 3150
@@
 $EndComp
 $Comp
-L Device:D_ALT D8
+L Device:LED_Filled D8
 U 1 1 5F413179
 P 14000 3150
@@
 $EndComp
 $Comp
-L Device:D_ALT D9
+L Device:LED_Filled D9
 U 1 1 5F43126B
 P 14200 3150
@@
 $EndComp
 $Comp
-L Device:D_ALT D10
+L Device:LED_Filled D10
 U 1 1 5F43127F
 P 14400 3150
@@
 $EndComp
 $Comp
-L Device:LED_ALT D11
+L Device:LED_Filled D11
 U 1 1 5F431293
 P 14600 3150
@@
 $EndComp
 $Comp
-L Device:LED_ALT D12
+L Device:LED_Filled D12
 U 1 1 5F4312A7
 P 14800 3150
@@
 $EndComp
 $Comp
-L Device:LED_ALT D13
+L Device:LED_Filled D13
 U 1 1 5F4312BB
 P 15000 3150
@@
 $EndComp
 $Comp
-L Device:LED_ALT D14
+L Device:LED_Filled D14
 U 1 1 5F4312CF
 P 15200 3150
@@
 $EndComp
 $Comp
-L Device:LED_ALT D15
+L Device:LED_Filled D15
 U 1 1 5F4312E3
 P 15400 3150
@@
 $EndComp
 $Comp
-L Device:LED_ALT D16
+L Device:LED_Filled D16
 U 1 1 5F4312F7
 P 15600 3150
@@
 	9450 5350 9450 5450
 $Comp
-L Device:D_ALT D17
+L Device:LED_Filled D17
 U 1 1 5FD25D31
 P 8000 7000
@@
 $EndComp
 $Comp
-L Device:D_ALT D18
+L Device:LED_Filled D18
 U 1 1 5FD25D45
 P 8200 7000
@@
 $EndComp
 $Comp
-L Device:D_ALT D19
+L Device:LED_Filled D19
 U 1 1 5FD25D59
 P 8400 7000
@@
 $EndComp
 $Comp
-L Device:D_ALT D20
+L Device:LED_Filled D20
 U 1 1 5FD25D6D
 P 8600 7000
@@
 $EndComp
 $Comp
-L Device:D_ALT D21
+L Device:LED_Filled D21
 U 1 1 5FD25D81
 P 8800 7000
@@
 $EndComp
 $Comp
-L Device:D_ALT D22
+L Device:LED_Filled D22
 U 1 1 5FD25D95
 P 9000 7000
@@
 $EndComp
 $Comp
-L Device:D_ALT D23
+L Device:LED_Filled D23
 U 1 1 5FD25DA9
 P 9200 7000
@@
 NoConn ~ 8850 5950
 $Comp
-L Device:CP1 C13
+L Device:C_Polarized_US C13
 U 1 1 6022740E
 P 13550 5600
@@
 $EndComp
 $Comp
-L Device:CP1 C14
+L Device:C_Polarized_US C14
 U 1 1 6026F09E
 P 13950 5600
